Commit message: feat: 양팔 로봇 자산 4종 라인업(dg5f-m/dg5f-s/rh56f1/gripper) + head_v1 + 실기 정합 파이프라인
- generate_rl_urdf: SOURCES 4종(그리퍼 양팔 소스는 tools/gen_gripper_bi_source.sh), head_v1(vendor/head_v1 ← tools/import_head_v1.py),
  body 벤더 하우징 제거·기둥 z 0.730 절단(crop_body_plate), 무질량/0질량 링크 1e-5 kg, DG-5F 손 1.763 kg(실측),
  manifest collision_approximation(OpenArm hull / 손 decomposition)·camera_view_frame.rgb_lens_usd_frame(ir_projector_frame).
- build_usd: 4종 ASSET_BUILDS(벤더 게인: arm control_gains, DG-5F PID, 그리퍼 5.0/0.1; RH56F1 PD 없음), 링크별 콜라이더 override,
  prismatic mimic, head_v1.usda 이식(graft_head_v1)+검증, build_trace.log(isaaclab.sh 가 종료코드를 삼킨다).
- gen_fabric_urdfs: 7 변형(dg5f-m/dg5f-s/gripper 좌우 + rh56f1), 실링크 관성 동기·palm lump·헬퍼 1e-5, DG-5F 좌 템플릿.
- 테스트 103, 픽스처는 tmp OUT_DIR(감사 필터쌍 보존). 구 자산 generated/rl/<old>/ 번들 삭제(URDF/manifest 는 동결 보관).

Co-Authored-By: Claude Fable 5.1 <noreply@anthropic.com>
Claude-Session: https://claude.ai/code/session_01B2gFUoGNzc6ZVktHojTXc7

File: eef/fabric_templates/openarm_tesollo_bi_s.urdf (robot description, URDF)
Before this commit: robot open_tesollo, 62 links, 61 joints
Links:
- link openarm: mass 0.001 -> 1e-05
- link openarm_right_link2_sphere2: mass 0.001 -> 1e-05
- link openarm_right_link2_sphere3: mass 0.001 -> 1e-05
- link openarm_right_link4_sphere2: mass 0.001 -> 1e-05
- link openarm_right_link4_sphere3: mass 0.001 -> 1e-05
- link openarm_right_link6_sphere2: mass 0.001 -> 1e-05
- link palm_center: mass 0.001 -> 1e-05
- link palm_link_sphere2: mass 0.001 -> 1e-05
- link palm_x: mass 0.001 -> 1e-05
- link palm_x_neg: mass 0.001 -> 1e-05
- link palm_y: mass 0.001 -> 1e-05
- link palm_y_neg: mass 0.001 -> 1e-05
- link palm_z: mass 0.001 -> 1e-05
- link palm_z_neg: mass 0.001 -> 1e-05
- link rl_dg_ee: mass 0.001 -> 1e-05
- link tesollo_right_rl_dg_1_1_sphere2: mass 0.001 -> 1e-05
- link tesollo_right_rl_dg_1_3_sphere2: mass 0.001 -> 1e-05
- link tesollo_right_rl_dg_2_1_sphere2: mass 0.001 -> 1e-05
- link tesollo_right_rl_dg_2_3_sphere2: mass 0.001 -> 1e-05
- link tesollo_right_rl_dg_3_1_sphere2: mass 0.001 -> 1e-05
- link tesollo_right_rl_dg_3_3_sphere2: mass 0.001 -> 1e-05
- link tesollo_right_rl_dg_4_1_sphere2: mass 0.001 -> 1e-05
- link tesollo_right_rl_dg_4_3_sphere2: mass 0.001 -> 1e-05
- link tesollo_right_rl_dg_5_1_sphere2: mass 0.001 -> 1e-05
- link tesollo_right_rl_dg_5_3_sphere2: mass 0.001 -> 1e-05
- link world_body_sphere1: mass 0.001 -> 1e-05
- link world_body_sphere2: mass 0.001 -> 1e-05
- link world_body_sphere3: mass 0.001 -> 1e-05

File: eef/fabric_templates/openarm_tesollo_bi_s_left.urdf (robot description, URDF)
Before this commit: robot openarm_tesollo_bi_s_left, 62 links, 61 joints
Links:
- link openarm: mass 0.001 -> 1e-05
- link openarm_right_link2_sphere2: mass 0.001 -> 1e-05
- link openarm_right_link2_sphere3: mass 0.001 -> 1e-05
- link openarm_right_link4_sphere2: mass 0.001 -> 1e-05
- link openarm_right_link4_sphere3: mass 0.001 -> 1e-05
- link openarm_right_link6_sphere2: mass 0.001 -> 1e-05
- link palm_center: mass 0.001 -> 1e-05
- link palm_link_sphere2: mass 0.001 -> 1e-05
- link palm_x: mass 0.001 -> 1e-05
- link palm_x_neg: mass 0.001 -> 1e-05
- link palm_y: mass 0.001 -> 1e-05
- link palm_y_neg: mass 0.001 -> 1e-05
- link palm_z: mass 0.001 -> 1e-05
- link palm_z_neg: mass 0.001 -> 1e-05
- link rl_dg_ee: mass 0.001 -> 1e-05
- link tesollo_right_rl_dg_1_1_sphere2: mass 0.001 -> 1e-05
- link tesollo_right_rl_dg_1_3_sphere2: mass 0.001 -> 1e-05
- link tesollo_right_rl_dg_2_1_sphere2: mass 0.001 -> 1e-05
- link tesollo_right_rl_dg_2_3_sphere2: mass 0.001 -> 1e-05
- link tesollo_right_rl_dg_3_1_sphere2: mass 0.001 -> 1e-05
- link tesollo_right_rl_dg_3_3_sphere2: mass 0.001 -> 1e-05
- link tesollo_right_rl_dg_4_1_sphere2: mass 0.001 -> 1e-05
- link tesollo_right_rl_dg_4_3_sphere2: mass 0.001 -> 1e-05
- link tesollo_right_rl_dg_5_1_sphere2: mass 0.001 -> 1e-05
- link tesollo_right_rl_dg_5_3_sphere2: mass 0.001 -> 1e-05
- link world_body_sphere1: mass 0.001 -> 1e-05
- link world_body_sphere2: mass 0.001 -> 1e-05
- link world_body_sphere3: mass 0.001 -> 1e-05

File: eef/fabric_templates/openarm_tesollo_sensor_left_gripper.urdf (robot description, URDF)
Before this commit: robot openarm_tesollo_sensor_left_gripper, 62 links, 61 joints
Links:
- link openarm: mass 0.001 -> 1e-05
- link openarm_right_link2_sphere2: mass 0.001 -> 1e-05
- link openarm_right_link2_sphere3: mass 0.001 -> 1e-05
- link openarm_right_link4_sphere2: mass 0.001 -> 1e-05
- link openarm_right_link4_sphere3: mass 0.001 -> 1e-05
- link openarm_right_link6_sphere2: mass 0.001 -> 1e-05
- link palm_center: mass 0.001 -> 1e-05
- link palm_link_sphere2: mass 0.001 -> 1e-05
- link palm_x: mass 0.001 -> 1e-05
- link palm_x_neg: mass 0.001 -> 1e-05
- link palm_y: mass 0.001 -> 1e-05
- link palm_y_neg: mass 0.001 -> 1e-05
- link palm_z: mass 0.001 -> 1e-05
- link palm_z_neg: mass 0.001 -> 1e-05
- link rl_dg_ee: mass 0.001 -> 1e-05
- link tesollo_right_rl_dg_1_1_sphere2: mass 0.001 -> 1e-05
- link tesollo_right_rl_dg_1_3_sphere2: mass 0.001 -> 1e-05
- link tesollo_right_rl_dg_2_1_sphere2: mass 0.001 -> 1e-05
- link tesollo_right_rl_dg_2_3_sphere2: mass 0.001 -> 1e-05
- link tesollo_right_rl_dg_3_1_sphere2: mass 0.001 -> 1e-05
- link tesollo_right_rl_dg_3_3_sphere2: mass 0.001 -> 1e-05
- link tesollo_right_rl_dg_4_1_sphere2: mass 0.001 -> 1e-05
- link tesollo_right_rl_dg_4_3_sphere2: mass 0.001 -> 1e-05
- link tesollo_right_rl_dg_5_1_sphere2: mass 0.001 -> 1e-05
- link tesollo_right_rl_dg_5_3_sphere2: mass 0.001 -> 1e-05
- link world_body_sphere1: mass 0.001 -> 1e-05
- link world_body_sphere2: mass 0.001 -> 1e-05
- link world_body_sphere3: mass 0.001 -> 1e-05

File: eef/fabric_templates/openarm_tesollo_sensor_right.urdf (robot description, URDF)
Before this commit: robot open_tesollo, 62 links, 61 joints
Links:
- link openarm: mass 0.001 -> 1e-05
- link openarm_right_link2_sphere2: mass 0.001 -> 1e-05
- link openarm_right_link2_sphere3: mass 0.001 -> 1e-05
- link openarm_right_link4_sphere2: mass 0.001 -> 1e-05
- link openarm_right_link4_sphere3: mass 0.001 -> 1e-05
- link openarm_right_link6_sphere2: mass 0.001 -> 1e-05
- link palm_center: mass 0.001 -> 1e-05
- link palm_link_sphere2: mass 0.001 -> 1e-05
- link palm_x: mass 0.001 -> 1e-05
- link palm_x_neg: mass 0.001 -> 1e-05
- link palm_y: mass 0.001 -> 1e-05
- link palm_y_neg: mass 0.001 -> 1e-05
- link palm_z: mass 0.001 -> 1e-05
- link palm_z_neg: mass 0.001 -> 1e-05
- link rl_dg_ee: mass 0.001 -> 1e-05
- link tesollo_right_rl_dg_1_1_sphere2: mass 0.001 -> 1e-05
- link tesollo_right_rl_dg_1_3_sphere2: mass 0.001 -> 1e-05
- link tesollo_right_rl_dg_2_1_sphere2: mass 0.001 -> 1e-05
- link tesollo_right_rl_dg_2_3_sphere2: mass 0.001 -> 1e-05
- link tesollo_right_rl_dg_3_1_sphere2: mass 0.001 -> 1e-05
- link tesollo_right_rl_dg_3_3_sphere2: mass 0.001 -> 1e-05
- link tesollo_right_rl_dg_4_1_sphere2: mass 0.001 -> 1e-05
- link tesollo_right_rl_dg_4_3_sphere2: mass 0.001 -> 1e-05
- link tesollo_right_rl_dg_5_1_sphere2: mass 0.001 -> 1e-05
- link tesollo_right_rl_dg_5_3_sphere2: mass 0.001 -> 1e-05
- link world_body_sphere1: mass 0.001 -> 1e-05
- link world_body_sphere2: mass 0.001 -> 1e-05
- link world_body_sphere3: mass 0.001 -> 1e-05

File: generated/rl/openarm_bi_rh56f1_rl.urdf (robot description, URDF)
Before this commit: robot openarm_bi_rh56f1_rl, 76 links, 75 joints
Links:
- link head_base: mass 0.109629 -> 0.063863; geometry collision mesh filename=file:///home/user/rl_ws/urdf/vendor/head_v1/meshes/collisio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 scale=1 1 1; visual mesh filename=file:///home/user/rl_ws/urdf/vendor/head_v1/meshes/visual/h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 scale=1 1 1
- link head_camera: mass 0.065101 -> 0.068074; geometry collision mesh filename=file:///home/user/rl_ws/urdf/vendor/head_v1/meshes/collisio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 scale=1 1 1; visual mesh filename=file:///home/user/rl_ws/urdf/vendor/head_v1/meshes/visual/h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 scale=1 1 1
- link head_mid: mass 0.017073 -> 0.024281; geometry collision mesh filename=file:///home/user/rl_ws/urdf/vendor/head_v1/meshes/collisio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 scale=1 1 1; visual mesh filename=file:///home/user/rl_ws/urdf/vendor/head_v1/meshes/visual/h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 scale=1 1 1
Joints:
- joint head_j_cam_view: origin xyz=0.0147 0.0145 0.0365 rpy=0 0 0 -> xyz=0.0115 9.6e-05 0.036327 rpy=0 0 0
- joint head_j_pan: limit lower=-1.5708 upper=1.5708 effort=1.0 velocity=6.0 -> lower=-1.570796 upper=1.570796 effort=1.0 velocity=6.0; origin xyz=0.0225 0 0.0385 rpy=0 0 0 -> xyz=0.022500 0.000034 0.035603 rpy=0 0 0
- joint head_j_tilt: origin xyz=0 -0.0145 0.0275 rpy=0 0 0 -> xyz=0.000000 -0.011580 0.030400 rpy=0 0 0

File: generated/rl/openarm_tesollo_bi_rl.urdf (robot description, URDF)
Before this commit: robot openarm_dual_tesollo_rl, 84 links, 83 joints
Links:
- link head_base: mass 0.109629 -> 0.063863; geometry collision mesh filename=file:///home/user/rl_ws/urdf/vendor/head_v1/meshes/collisio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 scale=1 1 1; visual mesh filename=file:///home/user/rl_ws/urdf/vendor/head_v1/meshes/visual/h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 scale=1 1 1
- link head_camera: mass 0.065101 -> 0.068074; geometry collision mesh filename=file:///home/user/rl_ws/urdf/vendor/head_v1/meshes/collisio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 scale=1 1 1; visual mesh filename=file:///home/user/rl_ws/urdf/vendor/head_v1/meshes/visual/h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 scale=1 1 1
- link head_mid: mass 0.017073 -> 0.024281; geometry collision mesh filename=file:///home/user/rl_ws/urdf/vendor/head_v1/meshes/collisio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 scale=1 1 1; visual mesh filename=file:///home/user/rl_ws/urdf/vendor/head_v1/meshes/visual/h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 scale=1 1 1
Joints:
- joint head_j_cam_view: origin xyz=0.0147 0.0145 0.0365 rpy=0 0 0 -> xyz=0.0115 9.6e-05 0.036327 rpy=0 0 0
- joint head_j_pan: limit lower=-1.5708 upper=1.5708 effort=1.0 velocity=6.0 -> lower=-1.570796 upper=1.570796 effort=1.0 velocity=6.0; origin xyz=0.0225 0 0.0385 rpy=0 0 0 -> xyz=0.022500 0.000034 0.035603 rpy=0 0 0
- joint head_j_tilt: origin xyz=0 -0.0145 0.0275 rpy=0 0 0 -> xyz=0.000000 -0.011580 0.030400 rpy=0 0 0

File: generated/rl/openarm_tesollo_bi_s_rl.urdf (robot description, URDF)
Before this commit: robot openarm_dual_tesollo_s_rl, 84 links, 83 joints
Links:
- link head_base: mass 0.109629 -> 0.063863; geometry collision mesh filename=file:///home/user/rl_ws/urdf/vendor/head_v1/meshes/collisio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 scale=1 1 1; visual mesh filename=file:///home/user/rl_ws/urdf/vendor/head_v1/meshes/visual/h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 scale=1 1 1
- link head_camera: mass 0.065101 -> 0.068074; geometry collision mesh filename=file:///home/user/rl_ws/urdf/vendor/head_v1/meshes/collisio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 scale=1 1 1; visual mesh filename=file:///home/user/rl_ws/urdf/vendor/head_v1/meshes/visual/h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 scale=1 1 1
- link head_mid: mass 0.017073 -> 0.024281; geometry collision mesh filename=file:///home/user/rl_ws/urdf/vendor/head_v1/meshes/collisio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 scale=1 1 1; visual mesh filename=file:///home/user/rl_ws/urdf/vendor/head_v1/meshes/visual/h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 scale=1 1 1
Joints:
- joint head_j_cam_view: origin xyz=0.0147 0.0145 0.0365 rpy=0 0 0 -> xyz=0.0115 9.6e-05 0.036327 rpy=0 0 0
- joint head_j_pan: limit lower=-1.5708 upper=1.5708 effort=1.0 velocity=6.0 -> lower=-1.570796 upper=1.570796 effort=1.0 velocity=6.0; origin xyz=0.0225 0 0.0385 rpy=0 0 0 -> xyz=0.022500 0.000034 0.035603 rpy=0 0 0
- joint head_j_tilt: origin xyz=0 -0.0145 0.0275 rpy=0 0 0 -> xyz=0.000000 -0.011580 0.030400 rpy=0 0 0

File: generated/rl/openarm_tesollo_sensor_rl.urdf (robot description, URDF)
Before this commit: robot openarm_tesollo_sensor_rl, 57 links, 56 joints
Links:
- link head_base: mass 0.109629 -> 0.063863; geometry collision mesh filename=file:///home/user/rl_ws/urdf/vendor/head_v1/meshes/collisio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 scale=1 1 1; visual mesh filename=file:///home/user/rl_ws/urdf/vendor/head_v1/meshes/visual/h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 scale=1 1 1
- link head_camera: mass 0.065101 -> 0.068074; geometry collision mesh filename=file:///home/user/rl_ws/urdf/vendor/head_v1/meshes/collisio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 scale=1 1 1; visual mesh filename=file:///home/user/rl_ws/urdf/vendor/head_v1/meshes/visual/h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 scale=1 1 1
- link head_mid: mass 0.017073 -> 0.024281; geometry collision mesh filename=file:///home/user/rl_ws/urdf/vendor/head_v1/meshes/collisio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 scale=1 1 1; visual mesh filename=file:///home/user/rl_ws/urdf/vendor/head_v1/meshes/visual/h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 scale=1 1 1
Joints:
- joint head_j_cam_view: origin xyz=0.0147 0.0145 0.0365 rpy=0 0 0 -> xyz=0.0115 9.6e-05 0.036327 rpy=0 0 0
- joint head_j_pan: limit lower=-1.5708 upper=1.5708 effort=1.0 velocity=6.0 -> lower=-1.570796 upper=1.570796 effort=1.0 velocity=6.0; origin xyz=0.0225 0 0.0385 rpy=0 0 0 -> xyz=0.022500 0.000034 0.035603 rpy=0 0 0
- joint head_j_tilt: origin xyz=0 -0.0145 0.0275 rpy=0 0 0 -> xyz=0.000000 -0.011580 0.030400 rpy=0 0 0

File: vendor/delto_m_ros2/dg5f_driver/urdf/dg5f_right_ros2_control.xacro (robot description, xacro)
@@ -83,4 +83,8 @@
             <state_interface name="position" />
             <state_interface name="velocity" />
+            <!-- 08.31 추가: 하드웨어(system_interface.cpp:406)가 이미 export 하는데
+                 여기 선언이 없어 controller_manager 가 무시하고 있었다. 발열 추적에
+                 필요하다 — 엄지 rj_dg_1_4 가 막힌 채 계속 밀어붙여 뜨거워진 이력. -->
+            <state_interface name="temperature" />
         </joint>
         <joint name="rj_dg_1_2">
@@ -88,4 +92,8 @@
             <state_interface name="position" />
             <state_interface name="velocity" />
+            <!-- 08.31 추가: 하드웨어(system_interface.cpp:406)가 이미 export 하는데
+                 여기 선언이 없어 controller_manager 가 무시하고 있었다. 발열 추적에
+                 필요하다 — 엄지 rj_dg_1_4 가 막힌 채 계속 밀어붙여 뜨거워진 이력. -->
+            <state_interface name="temperature" />
         </joint>
         <joint name="rj_dg_1_3">
@@ -93,4 +101,8 @@
             <state_interface name="position" />
             <state_interface name="velocity" />
+            <!-- 08.31 추가: 하드웨어(system_interface.cpp:406)가 이미 export 하는데
+                 여기 선언이 없어 controller_manager 가 무시하고 있었다. 발열 추적에
+                 필요하다 — 엄지 rj_dg_1_4 가 막힌 채 계속 밀어붙여 뜨거워진 이력. -->
+            <state_interface name="temperature" />
         </joint>
         <joint name="rj_dg_1_4">
@@ -98,4 +110,8 @@
             <state_interface name="position" />
             <state_interface name="velocity" />
+            <!-- 08.31 추가: 하드웨어(system_interface.cpp:406)가 이미 export 하는데
+                 여기 선언이 없어 controller_manager 가 무시하고 있었다. 발열 추적에
+                 필요하다 — 엄지 rj_dg_1_4 가 막힌 채 계속 밀어붙여 뜨거워진 이력. -->
+            <state_interface name="temperature" />
         </joint>
         <!-- Finger 2 joints -->
@@ -104,4 +120,8 @@
             <state_interface name="position" />
             <state_interface name="velocity" />
+            <!-- 08.31 추가: 하드웨어(system_interface.cpp:406)가 이미 export 하는데
+                 여기 선언이 없어 controller_manager 가 무시하고 있었다. 발열 추적에
+                 필요하다 — 엄지 rj_dg_1_4 가 막힌 채 계속 밀어붙여 뜨거워진 이력. -->
+            <state_interface name="temperature" />
         </joint>
         <joint name="rj_dg_2_2">
@@ -109,4 +129,8 @@
             <state_interface name="position" />
             <state_interface name="velocity" />
+            <!-- 08.31 추가: 하드웨어(system_interface.cpp:406)가 이미 export 하는데
+                 여기 선언이 없어 controller_manager 가 무시하고 있었다. 발열 추적에
+                 필요하다 — 엄지 rj_dg_1_4 가 막힌 채 계속 밀어붙여 뜨거워진 이력. -->
+            <state_interface name="temperature" />
         </joint>
         <joint name="rj_dg_2_3">
@@ -114,4 +138,8 @@
             <state_interface name="position" />
             <state_interface name="velocity" />
+            <!-- 08.31 추가: 하드웨어(system_interface.cpp:406)가 이미 export 하는데
+                 여기 선언이 없어 controller_manager 가 무시하고 있었다. 발열 추적에
+                 필요하다 — 엄지 rj_dg_1_4 가 막힌 채 계속 밀어붙여 뜨거워진 이력. -->
+            <state_interface name="temperature" />
         </joint>
         <joint name="rj_dg_2_4">
@@ -119,4 +147,8 @@
             <state_interface name="position" />
             <state_interface name="velocity" />
+            <!-- 08.31 추가: 하드웨어(system_interface.cpp:406)가 이미 export 하는데
+                 여기 선언이 없어 controller_manager 가 무시하고 있었다. 발열 추적에
+                 필요하다 — 엄지 rj_dg_1_4 가 막힌 채 계속 밀어붙여 뜨거워진 이력. -->
+            <state_interface name="temperature" />
         </joint>
         <!-- Finger 3 joints -->
@@ -125,4 +157,8 @@
             <state_interface name="position" />
             <state_interface name="velocity" />
+            <!-- 08.31 추가: 하드웨어(system_interface.cpp:406)가 이미 export 하는데
+                 여기 선언이 없어 controller_manager 가 무시하고 있었다. 발열 추적에
+                 필요하다 — 엄지 rj_dg_1_4 가 막힌 채 계속 밀어붙여 뜨거워진 이력. -->
+            <state_interface name="temperature" />
         </joint>
         <joint name="rj_dg_3_2">
@@ -130,4 +166,8 @@
             <state_interface name="position" />
             <state_interface name="velocity" />
+            <!-- 08.31 추가: 하드웨어(system_interface.cpp:406)가 이미 export 하는데
+                 여기 선언이 없어 controller_manager 가 무시하고 있었다. 발열 추적에
+                 필요하다 — 엄지 rj_dg_1_4 가 막힌 채 계속 밀어붙여 뜨거워진 이력. -->
+            <state_interface name="temperature" />
         </joint>
         <joint name="rj_dg_3_3">
@@ -135,4 +175,8 @@
             <state_interface name="position" />
             <state_interface name="velocity" />
+            <!-- 08.31 추가: 하드웨어(system_interface.cpp:406)가 이미 export 하는데
+                 여기 선언이 없어 controller_manager 가 무시하고 있었다. 발열 추적에
+                 필요하다 — 엄지 rj_dg_1_4 가 막힌 채 계속 밀어붙여 뜨거워진 이력. -->
+            <state_interface name="temperature" />
         </joint>
         <joint name="rj_dg_3_4">
@@ -140,4 +184,8 @@
             <state_interface name="position" />
             <state_interface name="velocity" />
+            <!-- 08.31 추가: 하드웨어(system_interface.cpp:406)가 이미 export 하는데
+                 여기 선언이 없어 controller_manager 가 무시하고 있었다. 발열 추적에
+                 필요하다 — 엄지 rj_dg_1_4 가 막힌 채 계속 밀어붙여 뜨거워진 이력. -->
+            <state_interface name="temperature" />
         </joint>
         <!-- Finger 4 joints -->
@@ -146,4 +194,8 @@
             <state_interface name="position" />
             <state_interface name="velocity" />
+            <!-- 08.31 추가: 하드웨어(system_interface.cpp:406)가 이미 export 하는데
+                 여기 선언이 없어 controller_manager 가 무시하고 있었다. 발열 추적에
+                 필요하다 — 엄지 rj_dg_1_4 가 막힌 채 계속 밀어붙여 뜨거워진 이력. -->
+            <state_interface name="temperature" />
         </joint>
         <joint name="rj_dg_4_2">
@@ -151,4 +203,8 @@
             <state_interface name="position" />
             <state_interface name="velocity" />
+            <!-- 08.31 추가: 하드웨어(system_interface.cpp:406)가 이미 export 하는데
+                 여기 선언이 없어 controller_manager 가 무시하고 있었다. 발열 추적에
+                 필요하다 — 엄지 rj_dg_1_4 가 막힌 채 계속 밀어붙여 뜨거워진 이력. -->
+            <state_interface name="temperature" />
         </joint>
         <joint name="rj_dg_4_3">
@@ -156,4 +212,8 @@
             <state_interface name="position" />
             <state_interface name="velocity" />
+            <!-- 08.31 추가: 하드웨어(system_interface.cpp:406)가 이미 export 하는데
+                 여기 선언이 없어 controller_manager 가 무시하고 있었다. 발열 추적에
+                 필요하다 — 엄지 rj_dg_1_4 가 막힌 채 계속 밀어붙여 뜨거워진 이력. -->
+            <state_interface name="temperature" />
         </joint>
         <joint name="rj_dg_4_4">
@@ -161,4 +221,8 @@
             <state_interface name="position" />
             <state_interface name="velocity" />
+            <!-- 08.31 추가: 하드웨어(system_interface.cpp:406)가 이미 export 하는데
+                 여기 선언이 없어 controller_manager 가 무시하고 있었다. 발열 추적에
+                 필요하다 — 엄지 rj_dg_1_4 가 막힌 채 계속 밀어붙여 뜨거워진 이력. -->
+            <state_interface name="temperature" />
         </joint>
         <!-- Finger 5 joints -->
@@ -167,4 +231,8 @@
             <state_interface name="position" />
             <state_interface name="velocity" />
+            <!-- 08.31 추가: 하드웨어(system_interface.cpp:406)가 이미 export 하는데
+                 여기 선언이 없어 controller_manager 가 무시하고 있었다. 발열 추적에
+                 필요하다 — 엄지 rj_dg_1_4 가 막힌 채 계속 밀어붙여 뜨거워진 이력. -->
+            <state_interface name="temperature" />
         </joint>
         <joint name="rj_dg_5_2">
@@ -172,4 +240,8 @@
             <state_interface name="position" />
             <state_interface name="velocity" />
+            <!-- 08.31 추가: 하드웨어(system_interface.cpp:406)가 이미 export 하는데
+                 여기 선언이 없어 controller_manager 가 무시하고 있었다. 발열 추적에
+                 필요하다 — 엄지 rj_dg_1_4 가 막힌 채 계속 밀어붙여 뜨거워진 이력. -->
+            <state_interface name="temperature" />
         </joint>
         <joint name="rj_dg_5_3">
@@ -177,4 +249,8 @@
             <state_interface name="position" />
             <state_interface name="velocity" />
+            <!-- 08.31 추가: 하드웨어(system_interface.cpp:406)가 이미 export 하는데
+                 여기 선언이 없어 controller_manager 가 무시하고 있었다. 발열 추적에
+                 필요하다 — 엄지 rj_dg_1_4 가 막힌 채 계속 밀어붙여 뜨거워진 이력. -->
+            <state_interface name="temperature" />
         </joint>
         <joint name="rj_dg_5_4">
@@ -182,4 +258,8 @@
             <state_interface name="position" />
             <state_interface name="velocity" />
+            <!-- 08.31 추가: 하드웨어(system_interface.cpp:406)가 이미 export 하는데
+                 여기 선언이 없어 controller_manager 가 무시하고 있었다. 발열 추적에
+                 필요하다 — 엄지 rj_dg_1_4 가 막힌 채 계속 밀어붙여 뜨거워진 이력. -->
+            <state_interface name="temperature" />
         </joint>
     </ros2_control>
