Commit message: chore(dg5f-m): 자산 재생성 — convex_hull + 프레임 제거 반영
tools/generate_rl_urdf.py + tools/build_usd.py --sync-hdgp 산출물.
링크 84 → 80, 우측 손 31 → 29, collision shape 731 → 75.

File: generated/rl/openarm_dg5f-m_bi_rl.urdf (robot description, URDF)
Before this commit: robot openarm_dg5f_m_bi_rl, 84 links, 83 joints
Links:
- removed link l_hl_mount
- removed link l_hl_palm_alias
- removed link r_hl_mount
- removed link r_hl_palm_alias
Joints:
- removed joint l_hj_mount
- removed joint l_hj_palm_alias
- removed joint r_hj_mount
- removed joint r_hj_palm_alias
- joint l_hj_adapter: origin xyz=0 0 0 rpy=0 0 0 -> xyz=0 0 0.0495 rpy=0 -0 1.5707964; parent l_hl_mount -> l_al_7
- joint l_hj_palm_ee: origin xyz=0.028 0 0.04 rpy=0 0 0 -> xyz=0.028 0 0.04 rpy=0 -0 0; parent l_hl_palm_alias -> l_hl_palm
- joint r_hj_adapter: origin xyz=0 0 0 rpy=0 0 0 -> xyz=0 3e-07 0.0495 rpy=0 -0 -1.5707964; parent r_hl_mount -> r_al_7
- joint r_hj_palm_ee: origin xyz=0.028 0 0.04 rpy=0 0 0 -> xyz=0.028 0 0.04 rpy=0 -0 0; parent r_hl_palm_alias -> r_hl_palm
