Commit message: refactor(urdf): 자산 생성 기본 골자를 벤더 검증 구성으로 — 새 로봇도 같은 규격
DG-5F-M 에 개별로 적용했던 것을 **파이프라인 기본값**으로 올린다. 새 로봇은 아무것도
선언하지 않아도 같은 구조로 만들어지고, 벗어나려면 사유를 남겨야 한다.

① collision 근사: 기본을 `convex_hull` 로 뒤집는다(구: decomposition 기본 + hull 예외).
   근거는 벤더 자신의 Isaac 변환 설정(vendor/delto_m_ros2/dg_isaacsim/.../config.yaml
   `collider_type: convex_hull`). decomposition 이 필요한 자산은 `COLLIDER_DEVIATIONS` 에
   **사유와 함께** 등록한다(빈 사유는 빌드 에러). 현재 예외 둘 — rh56f1(allowlist 의
   accept_raw 가 decomposition 전제), gripper(조는 파지 도구, hull 이면 개구·파지 대역 무효).
   ⇒ dg5f-m-short·dg5f-s 가 hull 로 통일됐다. rh56f1·gripper 는 불변.

② 관절한계: 자산마다 **선언 필수**(빈 dict 허용, 미등록은 빌드 에러).
   벤더 한계는 자기관통 없는 가동 범위를 보장하지 않는다 — `_3/_4` 는 두 사본이 똑같이
   ±1.5708(placeholder), `thumb_1` 하한은 손바닥을 0.67 mm 파고든다. "아직 안 쟀다"와
   "잴 필요가 없다"를 구분해 남기기 위한 강제다. 미측정 자산 4종은 `{}` 로 등록.

③ 주소용 프레임 제거: 이름 하드코딩 → **규칙**(`find_addressing_frames`).
   지오메트리 없음 + 들어오는 고정관절 1개 + 앞뒤 중 하나가 항등변환.
   이름으로 참조되는 프레임은 `KEEP_ADDRESSING_FRAMES` 가 보존한다(`*_hl_palm_ee`,
   `head_cam_view`). ⇒ dg5f-m-short·dg5f-s 도 84→80 링크가 됐다(이름 추가 없이).

문서: docs/ROBOT_ASSET_SPEC.md — DG-5F-M 골자를 "왜 그렇게 하는가" 중심으로 정리했다.
새 로봇 추가 체크리스트(§6)와 09.09 에 실제로 밟은 함정 6가지(§7)를 포함한다.
특히 §2-1 측정 방법: 이웃 관절을 극단에 고정한 채 재면 조합을 재는 것이고, 같은 손가락
2-hop 쌍을 빼면 한계를 정하는 쌍이 측정에서 빠진다(둘 다 09.09 에 답이 뒤집힌 사례).

테스트 137 passed(신규 계약 2: 관절한계 선언 강제 · 프레임 제거가 규칙인지·멱등인지).

File: generated/rl/openarm_dg5f-m-short_bi_rl.urdf (robot description, URDF)
Before this commit: robot openarm_dg5f_m_short_bi_rl, 84 links, 83 joints
Links:
- removed link l_hl_mount
- removed link l_hl_palm_alias
- removed link r_hl_mount
- removed link r_hl_palm_alias
Joints:
- removed joint l_hj_adapter
- removed joint l_hj_palm_alias
- removed joint r_hj_adapter
- removed joint r_hj_palm_alias
- joint l_hj_mount: child l_hl_mount -> l_hl_adapter
- joint l_hj_palm_ee: origin xyz=0.028 0 0.04 rpy=0 0 0 -> xyz=0.028 0 0.04 rpy=0 -0 0; parent l_hl_palm_alias -> l_hl_palm
- joint r_hj_mount: child r_hl_mount -> r_hl_adapter
- joint r_hj_palm_ee: origin xyz=0.028 0 0.04 rpy=0 0 0 -> xyz=0.028 0 0.04 rpy=0 -0 0; parent r_hl_palm_alias -> r_hl_palm

File: generated/rl/openarm_dg5f-s_bi_rl.urdf (robot description, URDF)
Before this commit: robot openarm_dg5f_s_bi_rl, 84 links, 83 joints
Links:
- removed link l_hl_mount
- removed link l_hl_palm_alias
- removed link r_hl_mount
- removed link r_hl_palm_alias
Joints:
- removed joint l_hj_adapter
- removed joint l_hj_palm_alias
- removed joint r_hj_adapter
- removed joint r_hj_palm_alias
- joint l_hj_mount: child l_hl_mount -> l_hl_adapter
- joint l_hj_palm_ee: origin xyz=0.028 0 0.04 rpy=0 0 0 -> xyz=0.028 0 0.04 rpy=0 -0 0; parent l_hl_palm_alias -> l_hl_palm
- joint r_hj_mount: child r_hl_mount -> r_hl_adapter
- joint r_hj_palm_ee: origin xyz=0.028 0 0.04 rpy=0 0 0 -> xyz=0.028 0 0.04 rpy=0 -0 0; parent r_hl_palm_alias -> r_hl_palm
