Commit message: feat: DG-5F 손 자산 기준을 벤더 Isaac Sim USD 로 전환
Tesollo 가 repo/tesollo/tesollo_model 에 자기 Isaac Sim 자산을 배포한다.
sim 물리값의 기준은 매뉴얼 PDF 가 아니라 이쪽이다(사용자 확정 09.10).

- effort   2.0 -> 7.5 N·m      (drive:angular:physics:maxForce, 전 변종 동일)
- velocity 7.854 -> pi rad/s   (physxJoint:maxJointVelocity 180 deg/s)
- middle_1 한계 ±30° -> ±25°   (physics:lower/upperLimit)
- dg5f-m-short / dg5f-s 를 None 에서 실제 표로 교체
  · short 는 표준과 한계 동일(실측 대조), dg5f-s 는 별개 손
    (엄지 회전 ±90°, 굽힘 126~130°)

tools/dump_joint_inertia.py 신설 — 빌드된 USD 에서
physics:JointEquivalentInertia 를 뽑아 <asset>_joint_inertia.json 으로 남긴다.
벤더가 드라이브 게인을 관성 비례(k=625·I, d=0.25·I, USD 각도 단위)로 주므로,
숫자를 베끼지 않고 규칙을 우리 자산 관성에 적용하기 위한 입력이다.

Co-Authored-By: Claude Opus 5 <noreply@anthropic.com>
Claude-Session: https://claude.ai/code/session_01X3UjBxvcdQMDLsryR8e6J6

File: generated/rl/openarm_dg5f-s_bi_rl.urdf (robot description, URDF)
Before this commit: robot openarm_dg5f_s_bi_rl, 80 links, 79 joints
Joints:
- joint l_hj_index_1: limit lower=-0.2617993877991494 upper=0.8377580409572782 effort=7.5 velocity=3.141592653589793 -> lower=-0.261799 upper=0.837758 effort=7.5 velocity=3.142
- joint l_hj_index_2: limit lower=0 upper=2.199114857512855 effort=7.5 velocity=3.141592653589793 -> lower=0 upper=2.19911 effort=7.5 velocity=3.142
- joint l_hj_index_3: limit lower=-1.5707963267948966 upper=1.5707963267948966 effort=7.5 velocity=3.141592653589793 -> lower=-1.5708 upper=1.5708 effort=7.5 velocity=3.142
- joint l_hj_index_4: limit lower=-1.5707963267948966 upper=1.5707963267948966 effort=7.5 velocity=3.141592653589793 -> lower=-1.5708 upper=1.5708 effort=7.5 velocity=3.142
- joint l_hj_middle_1: limit lower=-0.7330382858376184 upper=0.5759586531581288 effort=7.5 velocity=3.141592653589793 -> lower=-0.733038 upper=0.575959 effort=7.5 velocity=3.142
- joint l_hj_middle_2: limit lower=0 upper=2.2689280275926285 effort=7.5 velocity=3.141592653589793 -> lower=0 upper=2.26893 effort=7.5 velocity=3.142
- joint l_hj_middle_3: limit lower=-1.5707963267948966 upper=1.5707963267948966 effort=7.5 velocity=3.141592653589793 -> lower=-1.5708 upper=1.5708 effort=7.5 velocity=3.142
- joint l_hj_middle_4: limit lower=-1.5707963267948966 upper=1.5707963267948966 effort=7.5 velocity=3.141592653589793 -> lower=-1.5708 upper=1.5708 effort=7.5 velocity=3.142
- joint l_hj_pinky_1: limit lower=-1.0471975511965976 upper=0 effort=7.5 velocity=3.141592653589793 -> lower=-1.0472 upper=-0 effort=7.5 velocity=3.142
- joint l_hj_pinky_2: limit lower=-1.5707963267948966 upper=0.6457718232379019 effort=7.5 velocity=3.141592653589793 -> lower=-1.5708 upper=0.645772 effort=7.5 velocity=3.142
- joint l_hj_pinky_3: limit lower=-1.5707963267948966 upper=1.5707963267948966 effort=7.5 velocity=3.141592653589793 -> lower=-1.5708 upper=1.5708 effort=7.5 velocity=3.142
- joint l_hj_pinky_4: limit lower=-1.5707963267948966 upper=1.5707963267948966 effort=7.5 velocity=3.141592653589793 -> lower=-1.5708 upper=1.5708 effort=7.5 velocity=3.142
- joint l_hj_ring_1: limit lower=-0.8377580409572782 upper=0.20943951023931956 effort=7.5 velocity=3.141592653589793 -> lower=-0.837758 upper=0.20944 effort=7.5 velocity=3.142
- joint l_hj_ring_2: limit lower=0 upper=2.2165681500327987 effort=7.5 velocity=3.141592653589793 -> lower=0 upper=2.21657 effort=7.5 velocity=3.142
- joint l_hj_ring_3: limit lower=-1.5707963267948966 upper=1.5707963267948966 effort=7.5 velocity=3.141592653589793 -> lower=-1.5708 upper=1.5708 effort=7.5 velocity=3.142
- joint l_hj_ring_4: limit lower=-1.5707963267948966 upper=1.5707963267948966 effort=7.5 velocity=3.141592653589793 -> lower=-1.5708 upper=1.5708 effort=7.5 velocity=3.142
- joint l_hj_thumb_1: limit lower=-1.5707963267948966 upper=1.5707963267948966 effort=7.5 velocity=3.141592653589793 -> lower=-1.5708 upper=1.5708 effort=7.5 velocity=3.142
- joint l_hj_thumb_2: limit lower=0 upper=2.670353755551324 effort=7.5 velocity=3.141592653589793 -> lower=-0 upper=2.67035 effort=7.5 velocity=3.142
- joint l_hj_thumb_3: limit lower=-1.5707963267948966 upper=1.5707963267948966 effort=7.5 velocity=3.141592653589793 -> lower=-1.5708 upper=1.5708 effort=7.5 velocity=3.142
- joint l_hj_thumb_4: limit lower=-1.5707963267948966 upper=1.5707963267948966 effort=7.5 velocity=3.141592653589793 -> lower=-1.5708 upper=1.5708 effort=7.5 velocity=3.142
- joint r_hj_index_1: limit lower=-0.8377580409572782 upper=0.2617993877991494 effort=7.5 velocity=3.141592653589793 -> lower=-0.837758 upper=0.261799 effort=7.5 velocity=3.142
- joint r_hj_index_2: limit lower=0 upper=2.199114857512855 effort=7.5 velocity=3.141592653589793 -> lower=0 upper=2.19911 effort=7.5 velocity=3.142
- joint r_hj_index_3: limit lower=-1.5707963267948966 upper=1.5707963267948966 effort=7.5 velocity=3.141592653589793 -> lower=-1.5708 upper=1.5708 effort=7.5 velocity=3.142
- joint r_hj_index_4: limit lower=-1.5707963267948966 upper=1.5707963267948966 effort=7.5 velocity=3.141592653589793 -> lower=-1.5708 upper=1.5708 effort=7.5 velocity=3.142
- joint r_hj_middle_1: limit lower=-0.5759586531581288 upper=0.7330382858376184 effort=7.5 velocity=3.141592653589793 -> lower=-0.575959 upper=0.733038 effort=7.5 velocity=3.142
- joint r_hj_middle_2: limit lower=0 upper=2.2689280275926285 effort=7.5 velocity=3.141592653589793 -> lower=0 upper=2.26893 effort=7.5 velocity=3.142
- joint r_hj_middle_3: limit lower=-1.5707963267948966 upper=1.5707963267948966 effort=7.5 velocity=3.141592653589793 -> lower=-1.5708 upper=1.5708 effort=7.5 velocity=3.142
- joint r_hj_middle_4: limit lower=-1.5707963267948966 upper=1.5707963267948966 effort=7.5 velocity=3.141592653589793 -> lower=-1.5708 upper=1.5708 effort=7.5 velocity=3.142
- joint r_hj_pinky_1: limit lower=0 upper=1.0471975511965976 effort=7.5 velocity=3.141592653589793 -> lower=0 upper=1.0472 effort=7.5 velocity=3.142
- joint r_hj_pinky_2: limit lower=-0.6457718232379019 upper=1.5707963267948966 effort=7.5 velocity=3.141592653589793 -> lower=-0.645772 upper=1.5708 effort=7.5 velocity=3.142
- joint r_hj_pinky_3: limit lower=-1.5707963267948966 upper=1.5707963267948966 effort=7.5 velocity=3.141592653589793 -> lower=-1.5708 upper=1.5708 effort=7.5 velocity=3.142
- joint r_hj_pinky_4: limit lower=-1.5707963267948966 upper=1.5707963267948966 effort=7.5 velocity=3.141592653589793 -> lower=-1.5708 upper=1.5708 effort=7.5 velocity=3.142
- joint r_hj_ring_1: limit lower=-0.20943951023931956 upper=0.8377580409572782 effort=7.5 velocity=3.141592653589793 -> lower=-0.20944 upper=0.837758 effort=7.5 velocity=3.142
- joint r_hj_ring_2: limit lower=0 upper=2.2165681500327987 effort=7.5 velocity=3.141592653589793 -> lower=0 upper=2.21657 effort=7.5 velocity=3.142
- joint r_hj_ring_3: limit lower=-1.5707963267948966 upper=1.5707963267948966 effort=7.5 velocity=3.141592653589793 -> lower=-1.5708 upper=1.5708 effort=7.5 velocity=3.142
- joint r_hj_ring_4: limit lower=-1.5707963267948966 upper=1.5707963267948966 effort=7.5 velocity=3.141592653589793 -> lower=-1.5708 upper=1.5708 effort=7.5 velocity=3.142
- joint r_hj_thumb_1: limit lower=-1.5707963267948966 upper=1.5707963267948966 effort=7.5 velocity=3.141592653589793 -> lower=-1.5708 upper=1.5708 effort=7.5 velocity=3.142
- joint r_hj_thumb_2: limit lower=-2.670353755551324 upper=0 effort=7.5 velocity=3.141592653589793 -> lower=-2.67035 upper=0 effort=7.5 velocity=3.142
- joint r_hj_thumb_3: limit lower=-1.5707963267948966 upper=1.5707963267948966 effort=7.5 velocity=3.141592653589793 -> lower=-1.5708 upper=1.5708 effort=7.5 velocity=3.142
- joint r_hj_thumb_4: limit lower=-1.5707963267948966 upper=1.5707963267948966 effort=7.5 velocity=3.141592653589793 -> lower=-1.5708 upper=1.5708 effort=7.5 velocity=3.142

File: generated/rl/openarm_dg5f-s_bi_rl/openarm_dg5f-s_bi_rl.urdf (robot description, URDF)
Before this commit: robot openarm_dg5f_s_bi_rl, 84 links, 83 joints
Links:
- removed link l_hl_mount
- removed link l_hl_palm_alias
- removed link r_hl_mount
- removed link r_hl_palm_alias
Joints:
- removed joint l_hj_adapter
- removed joint l_hj_palm_alias
- removed joint r_hj_adapter
- removed joint r_hj_palm_alias
- joint l_hj_index_1: limit lower=-0.2617993877991494 upper=0.8377580409572782 effort=7.5 velocity=3.141592653589793 -> lower=-0.261799 upper=0.837758 effort=7.5 velocity=3.142
- joint l_hj_index_2: limit lower=0 upper=2.199114857512855 effort=7.5 velocity=3.141592653589793 -> lower=0 upper=2.19911 effort=7.5 velocity=3.142
- joint l_hj_index_3: limit lower=-1.5707963267948966 upper=1.5707963267948966 effort=7.5 velocity=3.141592653589793 -> lower=-1.5708 upper=1.5708 effort=7.5 velocity=3.142
- joint l_hj_index_4: limit lower=-1.5707963267948966 upper=1.5707963267948966 effort=7.5 velocity=3.141592653589793 -> lower=-1.5708 upper=1.5708 effort=7.5 velocity=3.142
- joint l_hj_middle_1: limit lower=-0.7330382858376184 upper=0.5759586531581288 effort=7.5 velocity=3.141592653589793 -> lower=-0.733038 upper=0.575959 effort=7.5 velocity=3.142
- joint l_hj_middle_2: limit lower=0 upper=2.2689280275926285 effort=7.5 velocity=3.141592653589793 -> lower=0 upper=2.26893 effort=7.5 velocity=3.142
- joint l_hj_middle_3: limit lower=-1.5707963267948966 upper=1.5707963267948966 effort=7.5 velocity=3.141592653589793 -> lower=-1.5708 upper=1.5708 effort=7.5 velocity=3.142
- joint l_hj_middle_4: limit lower=-1.5707963267948966 upper=1.5707963267948966 effort=7.5 velocity=3.141592653589793 -> lower=-1.5708 upper=1.5708 effort=7.5 velocity=3.142
- joint l_hj_mount: child l_hl_mount -> l_hl_adapter
- joint l_hj_palm_ee: origin xyz=0.028 0 0.04 rpy=0 0 0 -> xyz=0.028 0 0.04 rpy=0 -0 0; parent l_hl_palm_alias -> l_hl_palm
- joint l_hj_pinky_1: limit lower=-1.0471975511965976 upper=0 effort=7.5 velocity=3.141592653589793 -> lower=-1.0472 upper=-0 effort=7.5 velocity=3.142
- joint l_hj_pinky_2: limit lower=-1.5707963267948966 upper=0.6457718232379019 effort=7.5 velocity=3.141592653589793 -> lower=-1.5708 upper=0.645772 effort=7.5 velocity=3.142
- joint l_hj_pinky_3: limit lower=-1.5707963267948966 upper=1.5707963267948966 effort=7.5 velocity=3.141592653589793 -> lower=-1.5708 upper=1.5708 effort=7.5 velocity=3.142
- joint l_hj_pinky_4: limit lower=-1.5707963267948966 upper=1.5707963267948966 effort=7.5 velocity=3.141592653589793 -> lower=-1.5708 upper=1.5708 effort=7.5 velocity=3.142
- joint l_hj_ring_1: limit lower=-0.8377580409572782 upper=0.20943951023931956 effort=7.5 velocity=3.141592653589793 -> lower=-0.837758 upper=0.20944 effort=7.5 velocity=3.142
- joint l_hj_ring_2: limit lower=0 upper=2.2165681500327987 effort=7.5 velocity=3.141592653589793 -> lower=0 upper=2.21657 effort=7.5 velocity=3.142
- joint l_hj_ring_3: limit lower=-1.5707963267948966 upper=1.5707963267948966 effort=7.5 velocity=3.141592653589793 -> lower=-1.5708 upper=1.5708 effort=7.5 velocity=3.142
- joint l_hj_ring_4: limit lower=-1.5707963267948966 upper=1.5707963267948966 effort=7.5 velocity=3.141592653589793 -> lower=-1.5708 upper=1.5708 effort=7.5 velocity=3.142
- joint l_hj_thumb_1: limit lower=-1.5707963267948966 upper=1.5707963267948966 effort=7.5 velocity=3.141592653589793 -> lower=-1.5708 upper=1.5708 effort=7.5 velocity=3.142
- joint l_hj_thumb_2: limit lower=0 upper=2.670353755551324 effort=7.5 velocity=3.141592653589793 -> lower=-0 upper=2.67035 effort=7.5 velocity=3.142
- joint l_hj_thumb_3: limit lower=-1.5707963267948966 upper=1.5707963267948966 effort=7.5 velocity=3.141592653589793 -> lower=-1.5708 upper=1.5708 effort=7.5 velocity=3.142
- joint l_hj_thumb_4: limit lower=-1.5707963267948966 upper=1.5707963267948966 effort=7.5 velocity=3.141592653589793 -> lower=-1.5708 upper=1.5708 effort=7.5 velocity=3.142
- joint r_hj_index_1: limit lower=-0.8377580409572782 upper=0.2617993877991494 effort=7.5 velocity=3.141592653589793 -> lower=-0.837758 upper=0.261799 effort=7.5 velocity=3.142
- joint r_hj_index_2: limit lower=0 upper=2.199114857512855 effort=7.5 velocity=3.141592653589793 -> lower=0 upper=2.19911 effort=7.5 velocity=3.142
- joint r_hj_index_3: limit lower=-1.5707963267948966 upper=1.5707963267948966 effort=7.5 velocity=3.141592653589793 -> lower=-1.5708 upper=1.5708 effort=7.5 velocity=3.142
- joint r_hj_index_4: limit lower=-1.5707963267948966 upper=1.5707963267948966 effort=7.5 velocity=3.141592653589793 -> lower=-1.5708 upper=1.5708 effort=7.5 velocity=3.142
- joint r_hj_middle_1: limit lower=-0.5759586531581288 upper=0.7330382858376184 effort=7.5 velocity=3.141592653589793 -> lower=-0.575959 upper=0.733038 effort=7.5 velocity=3.142
- joint r_hj_middle_2: limit lower=0 upper=2.2689280275926285 effort=7.5 velocity=3.141592653589793 -> lower=0 upper=2.26893 effort=7.5 velocity=3.142
- joint r_hj_middle_3: limit lower=-1.5707963267948966 upper=1.5707963267948966 effort=7.5 velocity=3.141592653589793 -> lower=-1.5708 upper=1.5708 effort=7.5 velocity=3.142
- joint r_hj_middle_4: limit lower=-1.5707963267948966 upper=1.5707963267948966 effort=7.5 velocity=3.141592653589793 -> lower=-1.5708 upper=1.5708 effort=7.5 velocity=3.142
- joint r_hj_mount: child r_hl_mount -> r_hl_adapter
- joint r_hj_palm_ee: origin xyz=0.028 0 0.04 rpy=0 0 0 -> xyz=0.028 0 0.04 rpy=0 -0 0; parent r_hl_palm_alias -> r_hl_palm
- joint r_hj_pinky_1: limit lower=0 upper=1.0471975511965976 effort=7.5 velocity=3.141592653589793 -> lower=0 upper=1.0472 effort=7.5 velocity=3.142
- joint r_hj_pinky_2: limit lower=-0.6457718232379019 upper=1.5707963267948966 effort=7.5 velocity=3.141592653589793 -> lower=-0.645772 upper=1.5708 effort=7.5 velocity=3.142
- joint r_hj_pinky_3: limit lower=-1.5707963267948966 upper=1.5707963267948966 effort=7.5 velocity=3.141592653589793 -> lower=-1.5708 upper=1.5708 effort=7.5 velocity=3.142
- joint r_hj_pinky_4: limit lower=-1.5707963267948966 upper=1.5707963267948966 effort=7.5 velocity=3.141592653589793 -> lower=-1.5708 upper=1.5708 effort=7.5 velocity=3.142
- joint r_hj_ring_1: limit lower=-0.20943951023931956 upper=0.8377580409572782 effort=7.5 velocity=3.141592653589793 -> lower=-0.20944 upper=0.837758 effort=7.5 velocity=3.142
- joint r_hj_ring_2: limit lower=0 upper=2.2165681500327987 effort=7.5 velocity=3.141592653589793 -> lower=0 upper=2.21657 effort=7.5 velocity=3.142
- joint r_hj_ring_3: limit lower=-1.5707963267948966 upper=1.5707963267948966 effort=7.5 velocity=3.141592653589793 -> lower=-1.5708 upper=1.5708 effort=7.5 velocity=3.142
- joint r_hj_ring_4: limit lower=-1.5707963267948966 upper=1.5707963267948966 effort=7.5 velocity=3.141592653589793 -> lower=-1.5708 upper=1.5708 effort=7.5 velocity=3.142
- joint r_hj_thumb_1: limit lower=-1.5707963267948966 upper=1.5707963267948966 effort=7.5 velocity=3.141592653589793 -> lower=-1.5708 upper=1.5708 effort=7.5 velocity=3.142
- joint r_hj_thumb_2: limit lower=-2.670353755551324 upper=0 effort=7.5 velocity=3.141592653589793 -> lower=-2.67035 upper=0 effort=7.5 velocity=3.142
- joint r_hj_thumb_3: limit lower=-1.5707963267948966 upper=1.5707963267948966 effort=7.5 velocity=3.141592653589793 -> lower=-1.5708 upper=1.5708 effort=7.5 velocity=3.142
- joint r_hj_thumb_4: limit lower=-1.5707963267948966 upper=1.5707963267948966 effort=7.5 velocity=3.141592653589793 -> lower=-1.5708 upper=1.5708 effort=7.5 velocity=3.142
