Commit message: chore(dg5f-m): 자산 재생성 — thumb_1 ±0.16, 프레임 제거 규칙 정정

File: generated/fabric/openarm_dg5f-m-short_bi_left/openarm_dg5f-m-short_bi_left.urdf (robot description, URDF)
Before this commit: robot openarm_dg5f-s_bi_right, 62 links, 61 joints
Links:
- link openarm_right_link1: geometry collision mesh filename=../openarm_tesollo/meshes/openarm_right_link1_collision_mes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 scale=1. 1. 1.; visual mesh filename=../openarm_tesollo/meshes/openarm_right_link1_visual_mesh.o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 scale=1. 1. 1.
- link openarm_right_link2: geometry collision mesh filename=../openarm_tesollo/meshes/openarm_right_link2_collision_mes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 scale=1. 1. 1.; visual mesh filename=../openarm_tesollo/meshes/openarm_right_link2_visual_mesh.o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 scale=1. 1. 1.
- link openarm_right_link3: geometry collision mesh filename=../openarm_tesollo/meshes/openarm_right_link3_collision_mes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 scale=1. 1. 1.; visual mesh filename=../openarm_tesollo/meshes/openarm_right_link3_visual_mesh.o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 scale=1. 1. 1.
- link openarm_right_link4: geometry collision mesh filename=../openarm_tesollo/meshes/openarm_right_link4_collision_mes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 scale=1. 1. 1.; visual mesh filename=../openarm_tesollo/meshes/openarm_right_link4_visual_mesh.o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 scale=1. 1. 1.
- link openarm_right_link5: geometry collision mesh filename=../openarm_tesollo/meshes/openarm_right_link5_collision_mes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 scale=1. 1. 1.; visual mesh filename=../openarm_tesollo/meshes/openarm_right_link5_visual_mesh.o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 scale=1. 1. 1.
- link openarm_right_link6: geometry collision mesh filename=../openarm_tesollo/meshes/openarm_right_link6_collision_mes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 scale=1. 1. 1.; visual mesh filename=../openarm_tesollo/meshes/openarm_right_link6_visual_mesh.o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 scale=1. 1. 1.
- link openarm_right_link7: geometry collision mesh filename=../openarm_tesollo/meshes/openarm_right_link7_collision_mes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 scale=1. 1. 1.; visual mesh filename=../openarm_tesollo/meshes/openarm_right_link7_visual_mesh.o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 scale=1. 1. 1.
- link palm_link: mass 0.68158 -> 0.75721; geometry collision mesh filename=../openarm_tesollo/meshes/rl_dg_base_c_mesh.obj scale=1. 1. 1.; collision mesh filename=../openarm_tesollo/meshes/rl_dg_mount_c_mesh.obj scale=1. 1. 1.
- link rl_dg_1_tip: mass 0.00365660775 -> 0.005
- link rl_dg_2_tip: mass 0.0036566 -> 0.005
- link rl_dg_3_tip: mass 0.00365660775 -> 0.005
- link rl_dg_4_tip: mass 0.00365660775 -> 0.005
- link rl_dg_5_tip: mass 0.00365660775 -> 0.005
- link tesollo_right_rl_dg_1_1: mass 0.0198063639 -> 0.0482; geometry collision mesh filename=../openarm_tesollo/meshes/rl_dg_1_1_c_mesh.obj scale=1. 1. 1.; visual mesh filename=../openarm_tesollo/meshes/tesollo_right_rl_dg_1_1_visuals_r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 scale=1. 1. 1.
- link tesollo_right_rl_dg_1_2: mass 0.0280995688 -> 0.0164; geometry collision mesh filename=../openarm_tesollo/meshes/rl_dg_1_2_c_mesh.obj scale=1. 1. 1.; visual mesh filename=../openarm_tesollo/meshes/tesollo_right_rl_dg_1_2_visuals_r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 scale=1. 1. 1.
- link tesollo_right_rl_dg_1_3: mass 0.0234819984 -> 0.0362; geometry collision mesh filename=../openarm_tesollo/meshes/rl_dg_1_3_c_mesh.obj scale=1. 1. 1.; visual mesh filename=../openarm_tesollo/meshes/tesollo_right_rl_dg_1_3_visuals_r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 scale=1. 1. 1.
- link tesollo_right_rl_dg_1_4: mass 0.0256150237 -> 0.0505; geometry collision mesh filename=../openarm_tesollo/meshes/rl_dg_1_4_c_mesh.obj scale=1. 1. 1.; collision mesh filename=../openarm_tesollo/meshes/rl_dg_1_tip_c_mesh.obj scale=1. 1. 1.
- link tesollo_right_rl_dg_2_1: mass 0.0330237441 -> 0.0546; geometry collision mesh filename=../openarm_tesollo/meshes/rl_dg_2_1_c_mesh.obj scale=1. 1. 1.; visual mesh filename=../openarm_tesollo/meshes/tesollo_right_rl_dg_2_1_visuals_r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 scale=1. 1. 1.
- link tesollo_right_rl_dg_2_2: mass 0.0234819993 -> 0.0362; geometry collision mesh filename=../openarm_tesollo/meshes/rl_dg_2_2_c_mesh.obj scale=1. 1. 1.; visual mesh filename=../openarm_tesollo/meshes/tesollo_right_rl_dg_2_2_visuals_r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 scale=1. 1. 1.
- link tesollo_right_rl_dg_2_3: mass 0.0234819993 -> 0.0362; geometry collision mesh filename=../openarm_tesollo/meshes/rl_dg_2_3_c_mesh.obj scale=1. 1. 1.; visual mesh filename=../openarm_tesollo/meshes/tesollo_right_rl_dg_2_3_visuals_r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 scale=1. 1. 1.
- link tesollo_right_rl_dg_2_4: mass 0.0120970504 -> 0.0266; geometry collision mesh filename=../openarm_tesollo/meshes/rl_dg_2_4_c_mesh.obj scale=1. 1. 1.; collision mesh filename=../openarm_tesollo/meshes/rl_dg_2_tip_c_mesh.obj scale=1. 1. 1.
- link tesollo_right_rl_dg_3_1: mass 0.0330237441 -> 0.0526; geometry collision mesh filename=../openarm_tesollo/meshes/rl_dg_3_1_c_mesh.obj scale=1. 1. 1.; visual mesh filename=../openarm_tesollo/meshes/tesollo_right_rl_dg_3_1_visuals_r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 scale=1. 1. 1.
- link tesollo_right_rl_dg_3_2: mass 0.0234819993 -> 0.0362; geometry collision mesh filename=../openarm_tesollo/meshes/rl_dg_3_2_c_mesh.obj scale=1. 1. 1.; visual mesh filename=../openarm_tesollo/meshes/tesollo_right_rl_dg_3_2_visuals_r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 scale=1. 1. 1.
- link tesollo_right_rl_dg_3_3: mass 0.0234819993 -> 0.0362; geometry collision mesh filename=../openarm_tesollo/meshes/rl_dg_3_3_c_mesh.obj scale=1. 1. 1.; visual mesh filename=../openarm_tesollo/meshes/tesollo_right_rl_dg_3_3_visuals_r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 scale=1. 1. 1.
- link tesollo_right_rl_dg_3_4: mass 0.0120970504 -> 0.0266; geometry collision mesh filename=../openarm_tesollo/meshes/rl_dg_3_4_c_mesh.obj scale=1. 1. 1.; collision mesh filename=../openarm_tesollo/meshes/rl_dg_3_tip_c_mesh.obj scale=1. 1. 1.
- link tesollo_right_rl_dg_4_1: mass 0.0330237441 -> 0.0548; geometry collision mesh filename=../openarm_tesollo/meshes/rl_dg_4_1_c_mesh.obj scale=1. 1. 1.; visual mesh filename=../openarm_tesollo/meshes/tesollo_right_rl_dg_4_1_visuals_r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 scale=1. 1. 1.
- link tesollo_right_rl_dg_4_2: mass 0.0234819976 -> 0.0362; geometry collision mesh filename=../openarm_tesollo/meshes/rl_dg_4_2_c_mesh.obj scale=1. 1. 1.; visual mesh filename=../openarm_tesollo/meshes/tesollo_right_rl_dg_4_2_visuals_r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 scale=1. 1. 1.
- link tesollo_right_rl_dg_4_3: mass 0.0234819993 -> 0.0362; geometry collision mesh filename=../openarm_tesollo/meshes/rl_dg_4_3_c_mesh.obj scale=1. 1. 1.; visual mesh filename=../openarm_tesollo/meshes/tesollo_right_rl_dg_4_3_visuals_r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 scale=1. 1. 1.
- link tesollo_right_rl_dg_4_4: mass 0.0120970504 -> 0.0266; geometry collision mesh filename=../openarm_tesollo/meshes/rl_dg_4_4_c_mesh.obj scale=1. 1. 1.; collision mesh filename=../openarm_tesollo/meshes/rl_dg_4_tip_c_mesh.obj scale=1. 1. 1.
- link tesollo_right_rl_dg_5_1: mass 0.0714341385 -> 0.0744; geometry collision mesh filename=../openarm_tesollo/meshes/rl_dg_5_1_c_mesh.obj scale=1. 1. 1.; visual mesh filename=../openarm_tesollo/meshes/tesollo_right_rl_dg_5_1_visuals_r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 scale=1. 1. 1.
- link tesollo_right_rl_dg_5_2: mass 0.0144987731 -> 0.0164; geometry collision mesh filename=../openarm_tesollo/meshes/rl_dg_5_2_c_mesh.obj scale=1. 1. 1.; visual mesh filename=../openarm_tesollo/meshes/tesollo_right_rl_dg_5_2_visuals_r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 scale=1. 1. 1.
- link tesollo_right_rl_dg_5_3: mass 0.0234819993 -> 0.0362; geometry collision mesh filename=../openarm_tesollo/meshes/rl_dg_5_3_c_mesh.obj scale=1. 1. 1.; visual mesh filename=../openarm_tesollo/meshes/tesollo_right_rl_dg_5_3_visuals_r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 scale=1. 1. 1.
- link tesollo_right_rl_dg_5_4: mass 0.0256146777 -> 0.0505; geometry collision mesh filename=../openarm_tesollo/meshes/rl_dg_5_4_c_mesh.obj scale=1. 1. 1.; collision mesh filename=../openarm_tesollo/meshes/rl_dg_5_tip_c_mesh.obj scale=1. 1. 1.
- link world: geometry collision mesh filename=../openarm_tesollo/meshes/openarm_body_link0_collision_mesh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 scale=1. 1. 1.; collision mesh filename=../openarm_tesollo/meshes/openarm_left_link0_collision_mesh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 scale=1. 1. 1.
Joints:
- joint openarm_right_joint1: limit lower=-1.396263 upper=3.490659 effort=40. velocity=16.7546644 -> lower=-3.490659 upper=1.396263 effort=40. velocity=16.7546644; origin xyz=0 -0.0935 0.68999977 rpy=1.5708 0 0 -> xyz=0 0.0935 0.68999977 rpy=-1.5708 0 0
- joint openarm_right_joint2: limit lower=-0.174532673 upper=3.31612533 effort=40. velocity=16.7546644 -> lower=-3.31612533 upper=0.174532673 effort=40. velocity=16.7546644; origin xyz=-0.0301 0 0.06 rpy=1.57079633 0 0 -> xyz=-0.0301 0 0.06 rpy=-1.57079633 0 0
- joint openarm_right_joint7: axis 0 1 0 -> 0 -1 0
- joint openarm_right_link2_joint_sphere2: origin xyz=0. 0. 0.03 rpy=0. 0. 0. -> xyz=0 0 0.03 rpy=0 0 0
- joint openarm_right_link2_joint_sphere3: origin xyz=0. 0. 0.06 rpy=0. 0. 0. -> xyz=0 0 0.06 rpy=0 0 0
- joint openarm_right_link4_joint_sphere2: origin xyz=0. 0. 0.05 rpy=0. 0. 0. -> xyz=0 0 0.05 rpy=0 0 0
- joint openarm_right_link4_joint_sphere3: origin xyz=0. 0. 0.10 rpy=0. 0. 0. -> xyz=0 0 0.1 rpy=0 0 0
- joint openarm_right_link6_joint_sphere2: origin xyz=0. 0. 0.05 rpy=0. 0. 0. -> xyz=0 0 0.05 rpy=0 0 0
- joint palm_center_joint: origin xyz=0. 0.03 0.04 rpy=0. 0. 0. -> xyz=0 -0.03 0.04 rpy=0 0 0
- joint palm_link_joint: origin xyz=0 3e-07 0.0685 rpy=0. 0. -1.5707964 -> xyz=0 -3e-07 0.076 rpy=0 0 1.5707964
- joint palm_link_joint_sphere2: origin xyz=0. 0. 0.02 rpy=0. 0. 0. -> xyz=0 0 0.02 rpy=0 0 0
- joint rj_dg_1_1: axis 0 0 1 -> 1 0 0; limit lower=-1.57079633 upper=1.57079633 effort=7.5 velocity=3.1415927 -> lower=-1.34390352 upper=0.383972435 effort=7.5 velocity=3.1415927; origin xyz=0.0017 0.018 0.0298 rpy=1.5708 0 1.5708 -> xyz=-0.0162 -0.019 0.0128 rpy=0 0 0
- joint rj_dg_1_2: limit lower=-2.67035376 upper=0 effort=7.5 velocity=3.1415927 -> lower=-0 upper=2.70526034 effort=7.5 velocity=3.1415927; origin xyz=0 0 0.0262 rpy=-1.5708 0 0 -> xyz=0.04195 0 0 rpy=0 0 0
- joint rj_dg_1_3: axis 0 0 1 -> 1 0 0; origin xyz=0.0381 0 0 rpy=1.5708 0 0 -> xyz=0 -0.031 0 rpy=0 0 0
- joint rj_dg_1_4: axis 0 0 1 -> 1 0 0; origin xyz=0.0334 0 0 rpy=0 0 0 -> xyz=0 -0.0388 0 rpy=0 0 0
- joint rj_dg_2_1: axis 0 0 1 -> 1 0 0; limit lower=-0.837758041 upper=0.261799388 effort=7.5 velocity=3.1415927 -> lower=-0.34906585 upper=0.541052068 effort=7.5 velocity=3.1415927; origin xyz=0.0017 0.028 0.08365 rpy=3.1416 -1.5708 0 -> xyz=-0.0071 -0.027 0.0661 rpy=0 0 0
- joint rj_dg_2_2: axis 0 0 -1 -> 0 1 0; limit lower=0 upper=2.19911486 effort=7.5 velocity=3.1415927 -> lower=-0 upper=2.00712864 effort=7.5 velocity=3.1415927; origin xyz=0.02415 0 0.0126 rpy=-1.5708 0 0 -> xyz=0.01765 0 0.0265 rpy=0 0 0
- joint rj_dg_2_3: axis 0 0 1 -> 0 1 0; origin xyz=0.0334 0 0 rpy=3.1416 0 0 -> xyz=0 0 0.0388 rpy=0 0 0
- joint rj_dg_2_4: axis 0 0 1 -> 0 1 0; origin xyz=0.0334 0 0 rpy=0 0 0 -> xyz=0 0 0.0388 rpy=0 0 0
- joint rj_dg_3_1: axis 0 0 1 -> 1 0 0; limit lower=-0.575958653 upper=0.733038286 effort=7.5 velocity=3.1415927 -> lower=-0.436332313 upper=0.436332313 effort=7.5 velocity=3.1415927; origin xyz=0.0017 0.005 0.08865 rpy=3.1416 -1.5708 0 -> xyz=-0.0071 -0.0025 0.0701 rpy=0 0 0
- joint rj_dg_3_2: axis 0 0 -1 -> 0 1 0; limit lower=0 upper=2.26892803 effort=7.5 velocity=3.1415927 -> lower=0 upper=2.00712864 effort=7.5 velocity=3.1415927; origin xyz=0.02415 0 0.0126 rpy=-1.5708 0 0 -> xyz=0.01765 0 0.0265 rpy=0 0 0
- joint rj_dg_3_3: axis 0 0 1 -> 0 1 0; origin xyz=0.0334 0 0 rpy=3.1416 0 0 -> xyz=0 0 0.0388 rpy=0 0 0
- joint rj_dg_3_4: axis 0 0 1 -> 0 1 0; origin xyz=0.0334 0 0 rpy=0 0 0 -> xyz=0 0 0.0388 rpy=0 0 0
- joint rj_dg_4_1: axis 0 0 1 -> 1 0 0; limit lower=-0.20943951 upper=0.837758041 effort=7.5 velocity=3.1415927 -> lower=-0.558505361 upper=0.261799388 effort=7.5 velocity=3.1415927; origin xyz=0.0013 -0.018 0.08065 rpy=3.1416 -1.5708 0 -> xyz=-0.0071 0.022 0.0621 rpy=0 0 0
- joint rj_dg_4_2: axis 0 0 -1 -> 0 1 0; limit lower=0 upper=2.21656815 effort=7.5 velocity=3.1415927 -> lower=0 upper=1.91986218 effort=7.5 velocity=3.1415927; origin xyz=0.02415 0 0.0126 rpy=-1.5708 0 0 -> xyz=0.01765 0 0.0265 rpy=0 0 0
- joint rj_dg_4_3: axis 0 0 1 -> 0 1 0; origin xyz=0.0334 0 0 rpy=3.1416 0 0 -> xyz=0 0 0.0388 rpy=0 0 0
- joint rj_dg_4_4: axis 0 0 1 -> 0 1 0; origin xyz=0.0334 0 0 rpy=0 0 0 -> xyz=0 0 0.0388 rpy=0 0 0
- joint rj_dg_5_1: limit lower=0 upper=1.04719755 effort=7.5 velocity=3.1415927 -> lower=-1.04719755 upper=0 effort=7.5 velocity=3.1415927; origin xyz=0.013 -0.01805 0.0364 rpy=0 0 -1.5708 -> xyz=0.0103 0.0195 0.0182 rpy=0 0 0
- joint rj_dg_5_2: axis 0 0 1 -> 1 0 0; limit lower=-0.645771823 upper=1.57079633 effort=7.5 velocity=3.1415927 -> lower=-1.57079633 upper=0.261799388 effort=7.5 velocity=3.1415927; origin xyz=0.02445 0 0.0307 rpy=-1.5708 0 0 -> xyz=0 0.028 0.0381 rpy=0 0 0
- joint rj_dg_5_3: axis 0 0 1 -> 0 1 0; origin xyz=0 -0.0272 0 rpy=1.5708 0 -1.5708 -> xyz=0 0 0.031 rpy=0 0 0
- joint rj_dg_5_4: axis 0 0 1 -> 0 1 0; origin xyz=0.0334 0 0 rpy=0 0 0 -> xyz=0 0 0.0388 rpy=0 0 0
- joint rl_dg_1_tip_joint: origin xyz=0.0289 0 0 rpy=0 0 0 -> xyz=0 -0.0363 0 rpy=0 0 0
- joint rl_dg_2_tip_joint: origin xyz=0.018 0 0 rpy=0 0 0 -> xyz=0 0 0.0255 rpy=0 0 0
- joint rl_dg_3_tip_joint: origin xyz=0.018 0 0 rpy=0 0 0 -> xyz=0 0 0.0255 rpy=0 0 0
- joint rl_dg_4_tip_joint: origin xyz=0.018 0 0 rpy=0 0 0 -> xyz=0 0 0.0255 rpy=0 0 0
- joint rl_dg_5_tip_joint: origin xyz=0.0289 0 0 rpy=0 0 0 -> xyz=0 0 0.0363 rpy=0 0 0
- joint rl_dg_ee_joint: origin xyz=0.023 0. 0.13 rpy=1.5707963 3.1415927 1.5707963 -> xyz=0.023 0 0.13 rpy=1.57079635 -4.64102067e-08 1.57079635
- joint root_joint: origin xyz=0. 0. 0. rpy=0. 0. 0. -> xyz=0 0 0 rpy=0 0 0
- joint tesollo_right_rl_dg_1_1_joint_sphere2: origin xyz=0.02 0. 0. rpy=0. 0. 0. -> xyz=0.02 0 0 rpy=0 0 0
- joint tesollo_right_rl_dg_1_3_joint_sphere2: origin xyz=0. 0.02 0. rpy=0. 0. 0. -> xyz=0 -0.02 0 rpy=0 0 0
- joint tesollo_right_rl_dg_2_1_joint_sphere2: origin xyz=0.02 0. 0. rpy=0. 0. 0. -> xyz=0.02 0 0 rpy=0 0 0
- joint tesollo_right_rl_dg_2_3_joint_sphere2: origin xyz=0. 0. 0.02 rpy=0. 0. 0. -> xyz=0 0 0.02 rpy=0 0 0
- joint tesollo_right_rl_dg_3_1_joint_sphere2: origin xyz=0.02 0. 0. rpy=0. 0. 0. -> xyz=0.02 0 0 rpy=0 0 0
- joint tesollo_right_rl_dg_3_3_joint_sphere2: origin xyz=0. 0. 0.02 rpy=0. 0. 0. -> xyz=0 0 0.02 rpy=0 0 0
- joint tesollo_right_rl_dg_4_1_joint_sphere2: origin xyz=0.02 0. 0. rpy=0. 0. 0. -> xyz=0.02 0 0 rpy=0 0 0
- joint tesollo_right_rl_dg_4_3_joint_sphere2: origin xyz=0. 0. 0.02 rpy=0. 0. 0. -> xyz=0 0 0.02 rpy=0 0 0
- joint tesollo_right_rl_dg_5_1_joint_sphere2: origin xyz=0. 0. 0.02 rpy=0. 0. 0. -> xyz=0 0 0.02 rpy=0 0 0
- joint tesollo_right_rl_dg_5_3_joint_sphere2: origin xyz=0. 0. 0.02 rpy=0. 0. 0. -> xyz=0 0 0.02 rpy=0 0 0
- joint world_body_joint_sphere1: origin xyz=0. 0. 0.15 rpy=0. 0. 0. -> xyz=0 0 0.15 rpy=0 0 0
- joint world_body_joint_sphere2: origin xyz=0. 0. 0.45 rpy=0. 0. 0. -> xyz=0 0 0.45 rpy=0 0 0
- joint world_body_joint_sphere3: origin xyz=0. 0. 0.70 rpy=0. 0. 0. -> xyz=0 0 0.7 rpy=0 0 0

File: generated/fabric/openarm_dg5f-m-short_bi_right/openarm_dg5f-m-short_bi_right.urdf (robot description, URDF)
Before this commit: robot openarm_dg5f-s_bi_right, 62 links, 61 joints
Links:
- link palm_link: mass 0.68158 -> 0.75721
- link rl_dg_1_tip: mass 0.00365660775 -> 0.005
- link rl_dg_2_tip: mass 0.0036566 -> 0.005
- link rl_dg_3_tip: mass 0.00365660775 -> 0.005
- link rl_dg_4_tip: mass 0.00365660775 -> 0.005
- link rl_dg_5_tip: mass 0.00365660775 -> 0.005
- link tesollo_right_rl_dg_1_1: mass 0.0198063639 -> 0.0482
- link tesollo_right_rl_dg_1_2: mass 0.0280995688 -> 0.0164
- link tesollo_right_rl_dg_1_3: mass 0.0234819984 -> 0.0362
- link tesollo_right_rl_dg_1_4: mass 0.0256150237 -> 0.0505
- link tesollo_right_rl_dg_2_1: mass 0.0330237441 -> 0.0546
- link tesollo_right_rl_dg_2_2: mass 0.0234819993 -> 0.0362
- link tesollo_right_rl_dg_2_3: mass 0.0234819993 -> 0.0362
- link tesollo_right_rl_dg_2_4: mass 0.0120970504 -> 0.0266
- link tesollo_right_rl_dg_3_1: mass 0.0330237441 -> 0.0526
- link tesollo_right_rl_dg_3_2: mass 0.0234819993 -> 0.0362
- link tesollo_right_rl_dg_3_3: mass 0.0234819993 -> 0.0362
- link tesollo_right_rl_dg_3_4: mass 0.0120970504 -> 0.0266
- link tesollo_right_rl_dg_4_1: mass 0.0330237441 -> 0.0548
- link tesollo_right_rl_dg_4_2: mass 0.0234819976 -> 0.0362
- link tesollo_right_rl_dg_4_3: mass 0.0234819993 -> 0.0362
- link tesollo_right_rl_dg_4_4: mass 0.0120970504 -> 0.0266
- link tesollo_right_rl_dg_5_1: mass 0.0714341385 -> 0.0744
- link tesollo_right_rl_dg_5_2: mass 0.0144987731 -> 0.0164
- link tesollo_right_rl_dg_5_3: mass 0.0234819993 -> 0.0362
- link tesollo_right_rl_dg_5_4: mass 0.0256146777 -> 0.0505
Joints:
- joint palm_link_joint: origin xyz=0 3e-07 0.0685 rpy=0. 0. -1.5707964 -> xyz=0 3e-07 0.076 rpy=0. 0. -1.5707964
- joint rj_dg_1_1: axis 0 0 1 -> 1 0 0; limit lower=-1.57079633 upper=1.57079633 effort=7.5 velocity=3.1415927 -> lower=-0.383972435 upper=1.34390352 effort=7.5 velocity=3.1415927; origin xyz=0.0017 0.018 0.0298 rpy=1.5708 0 1.5708 -> xyz=-0.0162 0.019 0.0128 rpy=0 0 0
- joint rj_dg_1_2: limit lower=-2.67035376 upper=0 effort=7.5 velocity=3.1415927 -> lower=-2.70526034 upper=0 effort=7.5 velocity=3.1415927; origin xyz=0 0 0.0262 rpy=-1.5708 0 0 -> xyz=0.04195 0 0 rpy=0 0 0
- joint rj_dg_1_3: axis 0 0 1 -> 1 0 0; origin xyz=0.0381 0 0 rpy=1.5708 0 0 -> xyz=0 0.031 0 rpy=0 0 0
- joint rj_dg_1_4: axis 0 0 1 -> 1 0 0; origin xyz=0.0334 0 0 rpy=0 0 0 -> xyz=0 0.0388 0 rpy=0 0 0
- joint rj_dg_2_1: axis 0 0 1 -> 1 0 0; limit lower=-0.837758041 upper=0.261799388 effort=7.5 velocity=3.1415927 -> lower=-0.541052068 upper=0.34906585 effort=7.5 velocity=3.1415927; origin xyz=0.0017 0.028 0.08365 rpy=3.1416 -1.5708 0 -> xyz=-0.0071 0.027 0.0661 rpy=0 0 0
- joint rj_dg_2_2: axis 0 0 -1 -> 0 1 0; limit lower=0 upper=2.19911486 effort=7.5 velocity=3.1415927 -> lower=-0 upper=2.00712864 effort=7.5 velocity=3.1415927; origin xyz=0.02415 0 0.0126 rpy=-1.5708 0 0 -> xyz=0.01765 0 0.0265 rpy=0 0 0
- joint rj_dg_2_3: axis 0 0 1 -> 0 1 0; origin xyz=0.0334 0 0 rpy=3.1416 0 0 -> xyz=0 0 0.0388 rpy=0 0 0
- joint rj_dg_2_4: axis 0 0 1 -> 0 1 0; origin xyz=0.0334 0 0 rpy=0 0 0 -> xyz=0 0 0.0388 rpy=0 0 0
- joint rj_dg_3_1: axis 0 0 1 -> 1 0 0; limit lower=-0.575958653 upper=0.733038286 effort=7.5 velocity=3.1415927 -> lower=-0.436332313 upper=0.436332313 effort=7.5 velocity=3.1415927; origin xyz=0.0017 0.005 0.08865 rpy=3.1416 -1.5708 0 -> xyz=-0.0071 0.0025 0.0701 rpy=0 0 0
- joint rj_dg_3_2: axis 0 0 -1 -> 0 1 0; limit lower=0 upper=2.26892803 effort=7.5 velocity=3.1415927 -> lower=0 upper=2.00712864 effort=7.5 velocity=3.1415927; origin xyz=0.02415 0 0.0126 rpy=-1.5708 0 0 -> xyz=0.01765 0 0.0265 rpy=0 0 0
- joint rj_dg_3_3: axis 0 0 1 -> 0 1 0; origin xyz=0.0334 0 0 rpy=3.1416 0 0 -> xyz=0 0 0.0388 rpy=0 0 0
- joint rj_dg_3_4: axis 0 0 1 -> 0 1 0; origin xyz=0.0334 0 0 rpy=0 0 0 -> xyz=0 0 0.0388 rpy=0 0 0
- joint rj_dg_4_1: axis 0 0 1 -> 1 0 0; limit lower=-0.20943951 upper=0.837758041 effort=7.5 velocity=3.1415927 -> lower=-0.261799388 upper=0.558505361 effort=7.5 velocity=3.1415927; origin xyz=0.0013 -0.018 0.08065 rpy=3.1416 -1.5708 0 -> xyz=-0.0071 -0.022 0.0621 rpy=0 0 0
- joint rj_dg_4_2: axis 0 0 -1 -> 0 1 0; limit lower=0 upper=2.21656815 effort=7.5 velocity=3.1415927 -> lower=0 upper=1.91986218 effort=7.5 velocity=3.1415927; origin xyz=0.02415 0 0.0126 rpy=-1.5708 0 0 -> xyz=0.01765 0 0.0265 rpy=0 0 0
- joint rj_dg_4_3: axis 0 0 1 -> 0 1 0; origin xyz=0.0334 0 0 rpy=3.1416 0 0 -> xyz=0 0 0.0388 rpy=0 0 0
- joint rj_dg_4_4: axis 0 0 1 -> 0 1 0; origin xyz=0.0334 0 0 rpy=0 0 0 -> xyz=0 0 0.0388 rpy=0 0 0
- joint rj_dg_5_1: limit lower=0 upper=1.04719755 effort=7.5 velocity=3.1415927 -> lower=-0 upper=1.04719755 effort=7.5 velocity=3.1415927; origin xyz=0.013 -0.01805 0.0364 rpy=0 0 -1.5708 -> xyz=0.0103 -0.0195 0.0182 rpy=0 0 0
- joint rj_dg_5_2: axis 0 0 1 -> 1 0 0; limit lower=-0.645771823 upper=1.57079633 effort=7.5 velocity=3.1415927 -> lower=-0.261799388 upper=1.57079633 effort=7.5 velocity=3.1415927; origin xyz=0.02445 0 0.0307 rpy=-1.5708 0 0 -> xyz=0 -0.028 0.0381 rpy=0 0 0
- joint rj_dg_5_3: axis 0 0 1 -> 0 1 0; origin xyz=0 -0.0272 0 rpy=1.5708 0 -1.5708 -> xyz=0 0 0.031 rpy=0 0 0
- joint rj_dg_5_4: axis 0 0 1 -> 0 1 0; origin xyz=0.0334 0 0 rpy=0 0 0 -> xyz=0 0 0.0388 rpy=0 0 0
- joint rl_dg_1_tip_joint: origin xyz=0.0289 0 0 rpy=0 0 0 -> xyz=0 0.0363 0 rpy=0 0 0
- joint rl_dg_2_tip_joint: origin xyz=0.018 0 0 rpy=0 0 0 -> xyz=0 0 0.0255 rpy=0 0 0
- joint rl_dg_3_tip_joint: origin xyz=0.018 0 0 rpy=0 0 0 -> xyz=0 0 0.0255 rpy=0 0 0
- joint rl_dg_4_tip_joint: origin xyz=0.018 0 0 rpy=0 0 0 -> xyz=0 0 0.0255 rpy=0 0 0
- joint rl_dg_5_tip_joint: origin xyz=0.0289 0 0 rpy=0 0 0 -> xyz=0 0 0.0363 rpy=0 0 0

File: generated/fabric/openarm_dg5f-m_bi_left/openarm_dg5f-m_bi_left.urdf (robot description, URDF)
Before this commit: robot openarm_dg5f-m_bi_left, 62 links, 61 joints
Links:
- link palm_link: mass 0.8893775 -> 0.8893575
Joints:
- joint rj_dg_1_1: limit lower=-0.890117919 upper=0.383972435 effort=7.5 velocity=3.1415927 -> lower=-0.16 upper=0.16 effort=7.5 velocity=3.1415927

File: generated/fabric/openarm_dg5f-m_bi_right/openarm_dg5f-m_bi_right.urdf (robot description, URDF)
Before this commit: robot openarm_dg5f-m_bi_right, 62 links, 61 joints
Links:
- link palm_link: mass 0.8893775 -> 0.8893575
Joints:
- joint rj_dg_1_1: limit lower=-0.383972435 upper=0.890117919 effort=7.5 velocity=3.1415927 -> lower=-0.16 upper=0.16 effort=7.5 velocity=3.1415927

File: generated/fabric/openarm_dg5f-s_bi_left/openarm_dg5f-s_bi_left.urdf (robot description, URDF)
Before this commit: robot openarm_dg5f-s_bi_left, 62 links, 61 joints
Links:
- link palm_link: mass 0.681604335 -> 0.681584335
