Commit message: chore(dg5f-m): 자산 재생성 — thumb_1 ±0.16, 프레임 제거 규칙 정정

File: generated/rl/openarm_dg5f-m-short_bi_rl.urdf (robot description, URDF)
Before this commit: robot openarm_dg5f_m_bi_rl, 80 links, 79 joints
Links:
- added link l_hl_mount, mass 1e-05
- added link l_hl_palm_alias, mass 1e-05
- added link r_hl_mount, mass 1e-05
- added link r_hl_palm_alias, mass 1e-05
- link l_hl_adapter: mass 0.0523145 -> 0.0882; geometry visual mesh filename=file:///home/user/rl_ws/urdf/vendor/tesollo_model/dg5f/mesh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
- link l_hl_base: mass 0.470831 -> 0.1112; geometry collision mesh filename=file:///home/user/rl_ws/urdf/vendor/tesollo_model/dg5f/mesh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; visual mesh filename=file:///home/user/rl_ws/urdf/vendor/tesollo_model/dg5f/mesh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
- link l_hl_index_1: mass 0.0470831 -> 0.0546; geometry collision mesh filename=file:///home/user/rl_ws/urdf/vendor/tesollo_model/dg5f/mesh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; visual mesh filename=file:///home/user/rl_ws/urdf/vendor/tesollo_model/dg5f/mesh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
- link l_hl_index_2: mass 0.0470831 -> 0.0362; geometry collision mesh filename=file:///home/user/rl_ws/urdf/vendor/tesollo_model/dg5f/mesh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; visual mesh filename=file:///home/user/rl_ws/urdf/vendor/tesollo_model/dg5f/mesh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
- link l_hl_index_3: mass 0.0470831 -> 0.0362; geometry collision mesh filename=file:///home/user/rl_ws/urdf/vendor/tesollo_model/dg5f/mesh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; visual mesh filename=file:///home/user/rl_ws/urdf/vendor/tesollo_model/dg5f/mesh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
- link l_hl_index_4: mass 0.0261573 -> 0.0266; geometry collision mesh filename=file:///home/user/rl_ws/urdf/vendor/tesollo_model/dg5f/mesh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; visual mesh filename=file:///home/user/rl_ws/urdf/vendor/tesollo_model/dg5f/mesh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
- link l_hl_index_tip: mass 0.00523145 -> 0.005; geometry collision mesh filename=file:///home/user/rl_ws/urdf/vendor/tesollo_model/dg5f/mesh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; visual mesh filename=file:///home/user/rl_ws/urdf/vendor/tesollo_model/dg5f/mesh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
- link l_hl_middle_1: mass 0.0470831 -> 0.0526; geometry collision mesh filename=file:///home/user/rl_ws/urdf/vendor/tesollo_model/dg5f/mesh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; visual mesh filename=file:///home/user/rl_ws/urdf/vendor/tesollo_model/dg5f/mesh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
- link l_hl_middle_2: mass 0.0470831 -> 0.0362; geometry collision mesh filename=file:///home/user/rl_ws/urdf/vendor/tesollo_model/dg5f/mesh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; visual mesh filename=file:///home/user/rl_ws/urdf/vendor/tesollo_model/dg5f/mesh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
- link l_hl_middle_3: mass 0.0470831 -> 0.0362; geometry collision mesh filename=file:///home/user/rl_ws/urdf/vendor/tesollo_model/dg5f/mesh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; visual mesh filename=file:///home/user/rl_ws/urdf/vendor/tesollo_model/dg5f/mesh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
- link l_hl_middle_4: mass 0.0261573 -> 0.0266; geometry collision mesh filename=file:///home/user/rl_ws/urdf/vendor/tesollo_model/dg5f/mesh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; visual mesh filename=file:///home/user/rl_ws/urdf/vendor/tesollo_model/dg5f/mesh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
- link l_hl_middle_tip: mass 0.00523145 -> 0.005; geometry collision mesh filename=file:///home/user/rl_ws/urdf/vendor/tesollo_model/dg5f/mesh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; visual mesh filename=file:///home/user/rl_ws/urdf/vendor/tesollo_model/dg5f/mesh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
- link l_hl_palm: mass 0.366202 -> 0.5578; geometry collision mesh filename=file:///home/user/rl_ws/urdf/vendor/tesollo_model/dg5f/mesh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; visual mesh filename=file:///home/user/rl_ws/urdf/vendor/tesollo_model/dg5f/mesh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
- link l_hl_pinky_1: mass 0.057546 -> 0.0744; geometry collision mesh filename=file:///home/user/rl_ws/urdf/vendor/tesollo_model/dg5f/mesh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; visual mesh filename=file:///home/user/rl_ws/urdf/vendor/tesollo_model/dg5f/mesh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
- link l_hl_pinky_2: mass 0.0261573 -> 0.0164; geometry collision mesh filename=file:///home/user/rl_ws/urdf/vendor/tesollo_model/dg5f/mesh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; visual mesh filename=file:///home/user/rl_ws/urdf/vendor/tesollo_model/dg5f/mesh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
- link l_hl_pinky_3: mass 0.0470831 -> 0.0362; geometry collision mesh filename=file:///home/user/rl_ws/urdf/vendor/tesollo_model/dg5f/mesh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; visual mesh filename=file:///home/user/rl_ws/urdf/vendor/tesollo_model/dg5f/mesh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
- link l_hl_pinky_4: mass 0.0470831 -> 0.0505; geometry collision mesh filename=file:///home/user/rl_ws/urdf/vendor/tesollo_model/dg5f/mesh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; visual mesh filename=file:///home/user/rl_ws/urdf/vendor/tesollo_model/dg5f/mesh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
- link l_hl_pinky_tip: mass 0.00523145 -> 0.005; geometry collision mesh filename=file:///home/user/rl_ws/urdf/vendor/tesollo_model/dg5f/mesh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; visual mesh filename=file:///home/user/rl_ws/urdf/vendor/tesollo_model/dg5f/mesh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
- link l_hl_ring_1: mass 0.0470831 -> 0.0548; geometry collision mesh filename=file:///home/user/rl_ws/urdf/vendor/tesollo_model/dg5f/mesh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; visual mesh filename=file:///home/user/rl_ws/urdf/vendor/tesollo_model/dg5f/mesh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
- link l_hl_ring_2: mass 0.0470831 -> 0.0362; geometry collision mesh filename=file:///home/user/rl_ws/urdf/vendor/tesollo_model/dg5f/mesh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; visual mesh filename=file:///home/user/rl_ws/urdf/vendor/tesollo_model/dg5f/mesh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
- link l_hl_ring_3: mass 0.0470831 -> 0.0362; geometry collision mesh filename=file:///home/user/rl_ws/urdf/vendor/tesollo_model/dg5f/mesh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; visual mesh filename=file:///home/user/rl_ws/urdf/vendor/tesollo_model/dg5f/mesh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
- link l_hl_ring_4: mass 0.0261573 -> 0.0266; geometry collision mesh filename=file:///home/user/rl_ws/urdf/vendor/tesollo_model/dg5f/mesh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; visual mesh filename=file:///home/user/rl_ws/urdf/vendor/tesollo_model/dg5f/mesh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
- link l_hl_ring_tip: mass 0.00523145 -> 0.005; geometry collision mesh filename=file:///home/user/rl_ws/urdf/vendor/tesollo_model/dg5f/mesh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; visual mesh filename=file:///home/user/rl_ws/urdf/vendor/tesollo_model/dg5f/mesh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
- link l_hl_thumb_1: mass 0.0470831 -> 0.0482; geometry collision mesh filename=file:///home/user/rl_ws/urdf/vendor/tesollo_model/dg5f/mesh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; visual mesh filename=file:///home/user/rl_ws/urdf/vendor/tesollo_model/dg5f/mesh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
- link l_hl_thumb_2: mass 0.0261573 -> 0.0164; geometry collision mesh filename=file:///home/user/rl_ws/urdf/vendor/tesollo_model/dg5f/mesh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; visual mesh filename=file:///home/user/rl_ws/urdf/vendor/tesollo_model/dg5f/mesh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
- link l_hl_thumb_3: mass 0.0470831 -> 0.0362; geometry collision mesh filename=file:///home/user/rl_ws/urdf/vendor/tesollo_model/dg5f/mesh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; visual mesh filename=file:///home/user/rl_ws/urdf/vendor/tesollo_model/dg5f/mesh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
- link l_hl_thumb_4: mass 0.0470831 -> 0.0505; geometry collision mesh filename=file:///home/user/rl_ws/urdf/vendor/tesollo_model/dg5f/mesh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; visual mesh filename=file:///home/user/rl_ws/urdf/vendor/tesollo_model/dg5f/mesh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
- link l_hl_thumb_tip: mass 0.00523145 -> 0.005; geometry collision mesh filename=file:///home/user/rl_ws/urdf/vendor/tesollo_model/dg5f/mesh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; visual mesh filename=file:///home/user/rl_ws/urdf/vendor/tesollo_model/dg5f/mesh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
- link r_hl_adapter: mass 0.0523145 -> 0.0882; geometry visual mesh filename=file:///home/user/rl_ws/urdf/vendor/tesollo_model/dg5f/mesh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
- link r_hl_base: mass 0.470831 -> 0.1112; geometry collision mesh filename=file:///home/user/rl_ws/urdf/vendor/tesollo_model/dg5f/mesh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; visual mesh filename=file:///home/user/rl_ws/urdf/vendor/tesollo_model/dg5f/mesh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
- link r_hl_index_1: mass 0.0470831 -> 0.0546; geometry collision mesh filename=file:///home/user/rl_ws/urdf/vendor/tesollo_model/dg5f/mesh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; visual mesh filename=file:///home/user/rl_ws/urdf/vendor/tesollo_model/dg5f/mesh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
- link r_hl_index_2: mass 0.0470831 -> 0.0362; geometry collision mesh filename=file:///home/user/rl_ws/urdf/vendor/tesollo_model/dg5f/mesh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; visual mesh filename=file:///home/user/rl_ws/urdf/vendor/tesollo_model/dg5f/mesh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
- link r_hl_index_3: mass 0.0470831 -> 0.0362; geometry collision mesh filename=file:///home/user/rl_ws/urdf/vendor/tesollo_model/dg5f/mesh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; visual mesh filename=file:///home/user/rl_ws/urdf/vendor/tesollo_model/dg5f/mesh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
- link r_hl_index_4: mass 0.0261573 -> 0.0266; geometry collision mesh filename=file:///home/user/rl_ws/urdf/vendor/tesollo_model/dg5f/mesh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; visual mesh filename=file:///home/user/rl_ws/urdf/vendor/tesollo_model/dg5f/mesh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
- link r_hl_index_tip: mass 0.00523145 -> 0.005; geometry collision mesh filename=file:///home/user/rl_ws/urdf/vendor/tesollo_model/dg5f/mesh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; visual mesh filename=file:///home/user/rl_ws/urdf/vendor/tesollo_model/dg5f/mesh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
- link r_hl_middle_1: mass 0.0470831 -> 0.0526; geometry collision mesh filename=file:///home/user/rl_ws/urdf/vendor/tesollo_model/dg5f/mesh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; visual mesh filename=file:///home/user/rl_ws/urdf/vendor/tesollo_model/dg5f/mesh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
- link r_hl_middle_2: mass 0.0470831 -> 0.0362; geometry collision mesh filename=file:///home/user/rl_ws/urdf/vendor/tesollo_model/dg5f/mesh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; visual mesh filename=file:///home/user/rl_ws/urdf/vendor/tesollo_model/dg5f/mesh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
- link r_hl_middle_3: mass 0.0470831 -> 0.0362; geometry collision mesh filename=file:///home/user/rl_ws/urdf/vendor/tesollo_model/dg5f/mesh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; visual mesh filename=file:///home/user/rl_ws/urdf/vendor/tesollo_model/dg5f/mesh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
- link r_hl_middle_4: mass 0.0261573 -> 0.0266; geometry collision mesh filename=file:///home/user/rl_ws/urdf/vendor/tesollo_model/dg5f/mesh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; visual mesh filename=file:///home/user/rl_ws/urdf/vendor/tesollo_model/dg5f/mesh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
- link r_hl_middle_tip: mass 0.00523145 -> 0.005; geometry collision mesh filename=file:///home/user/rl_ws/urdf/vendor/tesollo_model/dg5f/mesh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; visual mesh filename=file:///home/user/rl_ws/urdf/vendor/tesollo_model/dg5f/mesh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
- link r_hl_palm: mass 0.366202 -> 0.5578; geometry collision mesh filename=file:///home/user/rl_ws/urdf/vendor/tesollo_model/dg5f/mesh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; visual mesh filename=file:///home/user/rl_ws/urdf/vendor/tesollo_model/dg5f/mesh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
- link r_hl_pinky_1: mass 0.057546 -> 0.0744; geometry collision mesh filename=file:///home/user/rl_ws/urdf/vendor/tesollo_model/dg5f/mesh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; visual mesh filename=file:///home/user/rl_ws/urdf/vendor/tesollo_model/dg5f/mesh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
- link r_hl_pinky_2: mass 0.0261573 -> 0.0164; geometry collision mesh filename=file:///home/user/rl_ws/urdf/vendor/tesollo_model/dg5f/mesh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; visual mesh filename=file:///home/user/rl_ws/urdf/vendor/tesollo_model/dg5f/mesh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
- link r_hl_pinky_3: mass 0.0470831 -> 0.0362; geometry collision mesh filename=file:///home/user/rl_ws/urdf/vendor/tesollo_model/dg5f/mesh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; visual mesh filename=file:///home/user/rl_ws/urdf/vendor/tesollo_model/dg5f/mesh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
- link r_hl_pinky_4: mass 0.0470831 -> 0.0505; geometry collision mesh filename=file:///home/user/rl_ws/urdf/vendor/tesollo_model/dg5f/mesh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; visual mesh filename=file:///home/user/rl_ws/urdf/vendor/tesollo_model/dg5f/mesh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
- link r_hl_pinky_tip: mass 0.00523145 -> 0.005; geometry collision mesh filename=file:///home/user/rl_ws/urdf/vendor/tesollo_model/dg5f/mesh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; visual mesh filename=file:///home/user/rl_ws/urdf/vendor/tesollo_model/dg5f/mesh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
- link r_hl_ring_1: mass 0.0470831 -> 0.0548; geometry collision mesh filename=file:///home/user/rl_ws/urdf/vendor/tesollo_model/dg5f/mesh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; visual mesh filename=file:///home/user/rl_ws/urdf/vendor/tesollo_model/dg5f/mesh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
- link r_hl_ring_2: mass 0.0470831 -> 0.0362; geometry collision mesh filename=file:///home/user/rl_ws/urdf/vendor/tesollo_model/dg5f/mesh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; visual mesh filename=file:///home/user/rl_ws/urdf/vendor/tesollo_model/dg5f/mesh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
- link r_hl_ring_3: mass 0.0470831 -> 0.0362; geometry collision mesh filename=file:///home/user/rl_ws/urdf/vendor/tesollo_model/dg5f/mesh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; visual mesh filename=file:///home/user/rl_ws/urdf/vendor/tesollo_model/dg5f/mesh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
- link r_hl_ring_4: mass 0.0261573 -> 0.0266; geometry collision mesh filename=file:///home/user/rl_ws/urdf/vendor/tesollo_model/dg5f/mesh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; visual mesh filename=file:///home/user/rl_ws/urdf/vendor/tesollo_model/dg5f/mesh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
- link r_hl_ring_tip: mass 0.00523145 -> 0.005; geometry collision mesh filename=file:///home/user/rl_ws/urdf/vendor/tesollo_model/dg5f/mesh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; visual mesh filename=file:///home/user/rl_ws/urdf/vendor/tesollo_model/dg5f/mesh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
- link r_hl_thumb_1: mass 0.0470831 -> 0.0482; geometry collision mesh filename=file:///home/user/rl_ws/urdf/vendor/tesollo_model/dg5f/mesh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; visual mesh filename=file:///home/user/rl_ws/urdf/vendor/tesollo_model/dg5f/mesh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
- link r_hl_thumb_2: mass 0.0261573 -> 0.0164; geometry collision mesh filename=file:///home/user/rl_ws/urdf/vendor/tesollo_model/dg5f/mesh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; visual mesh filename=file:///home/user/rl_ws/urdf/vendor/tesollo_model/dg5f/mesh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
- link r_hl_thumb_3: mass 0.0470831 -> 0.0362; geometry collision mesh filename=file:///home/user/rl_ws/urdf/vendor/tesollo_model/dg5f/mesh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; visual mesh filename=file:///home/user/rl_ws/urdf/vendor/tesollo_model/dg5f/mesh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
- link r_hl_thumb_4: mass 0.0470831 -> 0.0505; geometry collision mesh filename=file:///home/user/rl_ws/urdf/vendor/tesollo_model/dg5f/mesh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; visual mesh filename=file:///home/user/rl_ws/urdf/vendor/tesollo_model/dg5f/mesh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
- link r_hl_thumb_tip: mass 0.00523145 -> 0.005; geometry collision mesh filename=file:///home/user/rl_ws/urdf/vendor/tesollo_model/dg5f/mesh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; visual mesh filename=file:///home/user/rl_ws/urdf/vendor/tesollo_model/dg5f/mesh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
Joints:
- added joint l_hj_adapter: type fixed, parent l_hl_mount, child l_hl_adapter, origin xyz=0 0 0 rpy=0 0 0
- added joint l_hj_palm_alias: type fixed, parent l_hl_palm, child l_hl_palm_alias, origin xyz=0 0 0 rpy=0 0 0
- added joint r_hj_adapter: type fixed, parent r_hl_mount, child r_hl_adapter, origin xyz=0 0 0 rpy=0 0 0
- added joint r_hj_palm_alias: type fixed, parent r_hl_palm, child r_hl_palm_alias, origin xyz=0 0 0 rpy=0 0 0
- joint l_hj_base: origin xyz=0 0 0.004 rpy=0 0 0 -> xyz=0 0 0.0045 rpy=0 0 0
- joint l_hj_index_1: limit lower=-0.6108652381980153 upper=0.4188790204786391 effort=7.5 velocity=3.141592653589793 -> lower=-0.3490658503988659 upper=0.5410520681182421 effort=7.5 velocity=3.141592653589793
- joint l_hj_middle_1: limit lower=-0.6108652381980153 upper=0.6108652381980153 effort=7.5 velocity=3.141592653589793 -> lower=-0.4363323129985824 upper=0.4363323129985824 effort=7.5 velocity=3.141592653589793
- joint l_hj_middle_2: limit lower=-0.0 upper=1.9547687622336491 effort=7.5 velocity=3.141592653589793 -> lower=0.0 upper=2.007128639793479 effort=7.5 velocity=3.141592653589793
- joint l_hj_mount: child l_hl_adapter -> l_hl_mount
- joint l_hj_palm: origin xyz=0 0 0.0698 rpy=0 0 0 -> xyz=0 0 0.022 rpy=0 0 0
- joint l_hj_palm_ee: origin xyz=0.028 0 0.04 rpy=0 -0 0 -> xyz=0.028 0 0.04 rpy=0 0 0; parent l_hl_palm -> l_hl_palm_alias
- joint l_hj_pinky_1: limit lower=-1.0471975511965976 upper=0.017453292519943295 effort=7.5 velocity=3.141592653589793 -> lower=-1.0471975511965976 upper=0.0 effort=7.5 velocity=3.141592653589793
- joint l_hj_pinky_2: limit lower=-0.6108652381980153 upper=0.4188790204786391 effort=7.5 velocity=3.141592653589793 -> lower=-1.5707963267948966 upper=0.2617993877991494 effort=7.5 velocity=3.141592653589793
- joint l_hj_ring_1: limit lower=-0.4188790204786391 upper=0.6108652381980153 effort=7.5 velocity=3.141592653589793 -> lower=-0.5585053606381855 upper=0.2617993877991494 effort=7.5 velocity=3.141592653589793
- joint l_hj_ring_2: limit lower=-0.0 upper=1.9024088846738192 effort=7.5 velocity=3.141592653589793 -> lower=0.0 upper=1.9198621771937625 effort=7.5 velocity=3.141592653589793
- joint l_hj_thumb_1: limit lower=-0.16 upper=0.16 effort=7.5 velocity=3.141592653589793 -> lower=-1.3439035240356338 upper=0.3839724354387525 effort=7.5 velocity=3.141592653589793
- joint l_hj_thumb_2: limit lower=-0.0 upper=3.141592653589793 effort=7.5 velocity=3.141592653589793 -> lower=-0.0 upper=2.705260340591211 effort=7.5 velocity=3.141592653589793
- joint r_hj_base: origin xyz=0 0 0.004 rpy=0 0 0 -> xyz=0 0 0.0045 rpy=0 0 0
- joint r_hj_index_1: limit lower=-0.4188790204786391 upper=0.6108652381980153 effort=7.5 velocity=3.141592653589793 -> lower=-0.5410520681182421 upper=0.3490658503988659 effort=7.5 velocity=3.141592653589793
- joint r_hj_middle_1: limit lower=-0.6108652381980153 upper=0.6108652381980153 effort=7.5 velocity=3.141592653589793 -> lower=-0.4363323129985824 upper=0.4363323129985824 effort=7.5 velocity=3.141592653589793
- joint r_hj_middle_2: limit lower=-0.0 upper=1.9547687622336491 effort=7.5 velocity=3.141592653589793 -> lower=0.0 upper=2.007128639793479 effort=7.5 velocity=3.141592653589793
- joint r_hj_mount: child r_hl_adapter -> r_hl_mount
- joint r_hj_palm: origin xyz=0 0 0.0698 rpy=0 0 0 -> xyz=0 0 0.022 rpy=0 0 0
- joint r_hj_palm_ee: origin xyz=0.028 0 0.04 rpy=0 -0 0 -> xyz=0.028 0 0.04 rpy=0 0 0; parent r_hl_palm -> r_hl_palm_alias
- joint r_hj_pinky_1: limit lower=-0.017453292519943295 upper=1.0471975511965976 effort=7.5 velocity=3.141592653589793 -> lower=-0.0 upper=1.0471975511965976 effort=7.5 velocity=3.141592653589793
- joint r_hj_pinky_2: limit lower=-0.4188790204786391 upper=0.6108652381980153 effort=7.5 velocity=3.141592653589793 -> lower=-0.2617993877991494 upper=1.5707963267948966 effort=7.5 velocity=3.141592653589793
- joint r_hj_ring_1: limit lower=-0.6108652381980153 upper=0.4188790204786391 effort=7.5 velocity=3.141592653589793 -> lower=-0.2617993877991494 upper=0.5585053606381855 effort=7.5 velocity=3.141592653589793
- joint r_hj_ring_2: limit lower=-0.0 upper=1.9024088846738192 effort=7.5 velocity=3.141592653589793 -> lower=0.0 upper=1.9198621771937625 effort=7.5 velocity=3.141592653589793
- joint r_hj_thumb_1: limit lower=-0.16 upper=0.16 effort=7.5 velocity=3.141592653589793 -> lower=-0.3839724354387525 upper=1.3439035240356338 effort=7.5 velocity=3.141592653589793
- joint r_hj_thumb_2: limit lower=-3.141592653589793 upper=0.0 effort=7.5 velocity=3.141592653589793 -> lower=-2.705260340591211 upper=0.0 effort=7.5 velocity=3.141592653589793

File: generated/rl/openarm_dg5f-m_bi_rl/openarm_dg5f-m_bi_rl.urdf (robot description, URDF)
Before this commit: robot openarm_dg5f_m_bi_rl, 80 links, 79 joints
Joints:
- removed joint l_hj_adapter
- removed joint r_hj_adapter
- added joint l_hj_mount: type fixed, parent l_al_7, child l_hl_adapter, origin xyz=0 0 0.0495 rpy=0 0 1.5707964
- added joint r_hj_mount: type fixed, parent r_al_7, child r_hl_adapter, origin xyz=0 0.0000003 0.0495 rpy=0 0 -1.5707964
- joint l_hj_thumb_1: limit lower=-0.8901179185171081 upper=0.3839724354387525 effort=7.5 velocity=3.141592653589793 -> lower=-0.16 upper=0.16 effort=7.5 velocity=3.141592653589793
- joint r_hj_thumb_1: limit lower=-0.3839724354387525 upper=0.8901179185171081 effort=7.5 velocity=3.141592653589793 -> lower=-0.16 upper=0.16 effort=7.5 velocity=3.141592653589793
