Commit message: fix(dg5f-m): 자기관통 없는 관절한계로 축소 — 28관절
측정과 사용자 판단을 합친 최종 한계표. 기하 측정은 `_2`·`_1` 을 편 채 관절 하나씩만
굽혀 **분리**했고, 같은 손가락 안쪽 2-hop 쌍(`_2↔_4`, `_2↔tip` 등)을 포함했다 —
PhysX 자동 필터는 직접 연결된 부모-자식뿐이라 굴곡 한계를 정하는 건 이 쌍들이다.

① `_1` 5개 × 양손 → [−0.16, +0.16]  (사용자 확정: 벌림은 무조건 옆 손가락을 침범한다)
   엄지는 실측으로도 하한 −22.9° 가 베이스를 0.67 mm 관통. 리셋은 전부 0.
   ⚠pinky_1 은 외전이 아니라 Z-flex 라 성격이 다르다(주석에 분리 지점 표시).

② thumb_3/_4 → [0, 1.05]
   다른 관절을 편 채 `_3=_4` 를 훑은 실측: 0~1.05 rad 은 간극 0.15 mm 유지,
   **1.20 rad(68.8°)부터 tip↔palm 4.95 mm 관통**.

③ index/middle/ring/pinky `_3/_4` → [0, 1.5708]
   상한은 벤더값 유지 — 네 손가락은 ±90° 까지 굽혀도 간극 5.2~8.4 mm 가 남는다
   (최근접이 `_2↔palm` 고정 배치라 각도와 무관). 하한만 0 으로 내린다:
   액션 범위는 이미 override 로 0 이었지만 **물리 한계가 ±1.571 이라 접촉이 관절을
   음수로 밀 수 있었다**(c 시리즈 실측 index_3 −1.16 rad = 66° 뒤로 꺾임).

가드 정정: 리셋(영 자세)은 **닫힌 구간** 안이면 된다. 경계는 정상 — `_3/_4` 하한 0 이 의도다.

File: generated/fabric/openarm_dg5f-m_bi_left/openarm_dg5f-m_bi_left.urdf (robot description, URDF)
Before this commit: robot openarm_dg5f-m_bi_left, 62 links, 61 joints
Joints:
- joint rj_dg_1_3: limit lower=-1.57079633 upper=1.57079633 effort=7.5 velocity=3.1415927 -> lower=0 upper=1.05 effort=7.5 velocity=3.1415927
- joint rj_dg_1_4: limit lower=-1.57079633 upper=1.57079633 effort=7.5 velocity=3.1415927 -> lower=0 upper=1.05 effort=7.5 velocity=3.1415927
- joint rj_dg_2_1: limit lower=-0.610865238 upper=0.41887902 effort=7.5 velocity=3.1415927 -> lower=-0.16 upper=0.16 effort=7.5 velocity=3.1415927
- joint rj_dg_2_3: limit lower=-1.57079633 upper=1.57079633 effort=7.5 velocity=3.1415927 -> lower=0 upper=1.5708 effort=7.5 velocity=3.1415927
- joint rj_dg_2_4: limit lower=-1.57079633 upper=1.57079633 effort=7.5 velocity=3.1415927 -> lower=0 upper=1.5708 effort=7.5 velocity=3.1415927
- joint rj_dg_3_1: limit lower=-0.610865238 upper=0.610865238 effort=7.5 velocity=3.1415927 -> lower=-0.16 upper=0.16 effort=7.5 velocity=3.1415927
- joint rj_dg_3_3: limit lower=-1.57079633 upper=1.57079633 effort=7.5 velocity=3.1415927 -> lower=0 upper=1.5708 effort=7.5 velocity=3.1415927
- joint rj_dg_3_4: limit lower=-1.57079633 upper=1.57079633 effort=7.5 velocity=3.1415927 -> lower=0 upper=1.5708 effort=7.5 velocity=3.1415927
- joint rj_dg_4_1: limit lower=-0.41887902 upper=0.610865238 effort=7.5 velocity=3.1415927 -> lower=-0.16 upper=0.16 effort=7.5 velocity=3.1415927
- joint rj_dg_4_3: limit lower=-1.57079633 upper=1.57079633 effort=7.5 velocity=3.1415927 -> lower=0 upper=1.5708 effort=7.5 velocity=3.1415927
- joint rj_dg_4_4: limit lower=-1.57079633 upper=1.57079633 effort=7.5 velocity=3.1415927 -> lower=0 upper=1.5708 effort=7.5 velocity=3.1415927
- joint rj_dg_5_1: limit lower=-1.04719755 upper=0.0174532925 effort=7.5 velocity=3.1415927 -> lower=-0.16 upper=0.0174533 effort=7.5 velocity=3.1415927
- joint rj_dg_5_3: limit lower=-1.57079633 upper=1.57079633 effort=7.5 velocity=3.1415927 -> lower=0 upper=1.5708 effort=7.5 velocity=3.1415927
- joint rj_dg_5_4: limit lower=-1.57079633 upper=1.57079633 effort=7.5 velocity=3.1415927 -> lower=0 upper=1.5708 effort=7.5 velocity=3.1415927

File: generated/fabric/openarm_dg5f-m_bi_right/openarm_dg5f-m_bi_right.urdf (robot description, URDF)
Before this commit: robot openarm_dg5f-m_bi_right, 62 links, 61 joints
Joints:
- joint rj_dg_1_3: limit lower=-1.57079633 upper=1.57079633 effort=7.5 velocity=3.1415927 -> lower=0 upper=1.05 effort=7.5 velocity=3.1415927
- joint rj_dg_1_4: limit lower=-1.57079633 upper=1.57079633 effort=7.5 velocity=3.1415927 -> lower=0 upper=1.05 effort=7.5 velocity=3.1415927
- joint rj_dg_2_1: limit lower=-0.41887902 upper=0.610865238 effort=7.5 velocity=3.1415927 -> lower=-0.16 upper=0.16 effort=7.5 velocity=3.1415927
- joint rj_dg_2_3: limit lower=-1.57079633 upper=1.57079633 effort=7.5 velocity=3.1415927 -> lower=0 upper=1.5708 effort=7.5 velocity=3.1415927
- joint rj_dg_2_4: limit lower=-1.57079633 upper=1.57079633 effort=7.5 velocity=3.1415927 -> lower=0 upper=1.5708 effort=7.5 velocity=3.1415927
- joint rj_dg_3_1: limit lower=-0.610865238 upper=0.610865238 effort=7.5 velocity=3.1415927 -> lower=-0.16 upper=0.16 effort=7.5 velocity=3.1415927
- joint rj_dg_3_3: limit lower=-1.57079633 upper=1.57079633 effort=7.5 velocity=3.1415927 -> lower=0 upper=1.5708 effort=7.5 velocity=3.1415927
- joint rj_dg_3_4: limit lower=-1.57079633 upper=1.57079633 effort=7.5 velocity=3.1415927 -> lower=0 upper=1.5708 effort=7.5 velocity=3.1415927
- joint rj_dg_4_1: limit lower=-0.610865238 upper=0.41887902 effort=7.5 velocity=3.1415927 -> lower=-0.16 upper=0.16 effort=7.5 velocity=3.1415927
- joint rj_dg_4_3: limit lower=-1.57079633 upper=1.57079633 effort=7.5 velocity=3.1415927 -> lower=0 upper=1.5708 effort=7.5 velocity=3.1415927
- joint rj_dg_4_4: limit lower=-1.57079633 upper=1.57079633 effort=7.5 velocity=3.1415927 -> lower=0 upper=1.5708 effort=7.5 velocity=3.1415927
- joint rj_dg_5_1: limit lower=-0.0174532925 upper=1.04719755 effort=7.5 velocity=3.1415927 -> lower=-0.0174533 upper=0.16 effort=7.5 velocity=3.1415927
- joint rj_dg_5_3: limit lower=-1.57079633 upper=1.57079633 effort=7.5 velocity=3.1415927 -> lower=0 upper=1.5708 effort=7.5 velocity=3.1415927
- joint rj_dg_5_4: limit lower=-1.57079633 upper=1.57079633 effort=7.5 velocity=3.1415927 -> lower=0 upper=1.5708 effort=7.5 velocity=3.1415927

File: generated/rl/openarm_dg5f-m_bi_rl.urdf (robot description, URDF)
Before this commit: robot openarm_dg5f_m_bi_rl, 80 links, 79 joints
Joints:
- joint l_hj_index_1: limit lower=-0.6108652381980153 upper=0.4188790204786391 effort=7.5 velocity=3.141592653589793 -> lower=-0.16 upper=0.16 effort=7.5 velocity=3.141592653589793
- joint l_hj_index_3: limit lower=-1.5707963267948966 upper=1.5707963267948966 effort=7.5 velocity=3.141592653589793 -> lower=0 upper=1.5708 effort=7.5 velocity=3.141592653589793
- joint l_hj_index_4: limit lower=-1.5707963267948966 upper=1.5707963267948966 effort=7.5 velocity=3.141592653589793 -> lower=0 upper=1.5708 effort=7.5 velocity=3.141592653589793
- joint l_hj_middle_1: limit lower=-0.6108652381980153 upper=0.6108652381980153 effort=7.5 velocity=3.141592653589793 -> lower=-0.16 upper=0.16 effort=7.5 velocity=3.141592653589793
- joint l_hj_middle_3: limit lower=-1.5707963267948966 upper=1.5707963267948966 effort=7.5 velocity=3.141592653589793 -> lower=0 upper=1.5708 effort=7.5 velocity=3.141592653589793
- joint l_hj_middle_4: limit lower=-1.5707963267948966 upper=1.5707963267948966 effort=7.5 velocity=3.141592653589793 -> lower=0 upper=1.5708 effort=7.5 velocity=3.141592653589793
- joint l_hj_pinky_1: limit lower=-1.0471975511965976 upper=0.017453292519943295 effort=7.5 velocity=3.141592653589793 -> lower=-0.16 upper=0.0174533 effort=7.5 velocity=3.141592653589793
- joint l_hj_pinky_3: limit lower=-1.5707963267948966 upper=1.5707963267948966 effort=7.5 velocity=3.141592653589793 -> lower=0 upper=1.5708 effort=7.5 velocity=3.141592653589793
- joint l_hj_pinky_4: limit lower=-1.5707963267948966 upper=1.5707963267948966 effort=7.5 velocity=3.141592653589793 -> lower=0 upper=1.5708 effort=7.5 velocity=3.141592653589793
- joint l_hj_ring_1: limit lower=-0.4188790204786391 upper=0.6108652381980153 effort=7.5 velocity=3.141592653589793 -> lower=-0.16 upper=0.16 effort=7.5 velocity=3.141592653589793
- joint l_hj_ring_3: limit lower=-1.5707963267948966 upper=1.5707963267948966 effort=7.5 velocity=3.141592653589793 -> lower=0 upper=1.5708 effort=7.5 velocity=3.141592653589793
- joint l_hj_ring_4: limit lower=-1.5707963267948966 upper=1.5707963267948966 effort=7.5 velocity=3.141592653589793 -> lower=0 upper=1.5708 effort=7.5 velocity=3.141592653589793
- joint l_hj_thumb_3: limit lower=-1.5707963267948966 upper=1.5707963267948966 effort=7.5 velocity=3.141592653589793 -> lower=0 upper=1.05 effort=7.5 velocity=3.141592653589793
- joint l_hj_thumb_4: limit lower=-1.5707963267948966 upper=1.5707963267948966 effort=7.5 velocity=3.141592653589793 -> lower=0 upper=1.05 effort=7.5 velocity=3.141592653589793
- joint r_hj_index_1: limit lower=-0.4188790204786391 upper=0.6108652381980153 effort=7.5 velocity=3.141592653589793 -> lower=-0.16 upper=0.16 effort=7.5 velocity=3.141592653589793
- joint r_hj_index_3: limit lower=-1.5707963267948966 upper=1.5707963267948966 effort=7.5 velocity=3.141592653589793 -> lower=0 upper=1.5708 effort=7.5 velocity=3.141592653589793
- joint r_hj_index_4: limit lower=-1.5707963267948966 upper=1.5707963267948966 effort=7.5 velocity=3.141592653589793 -> lower=0 upper=1.5708 effort=7.5 velocity=3.141592653589793
- joint r_hj_middle_1: limit lower=-0.6108652381980153 upper=0.6108652381980153 effort=7.5 velocity=3.141592653589793 -> lower=-0.16 upper=0.16 effort=7.5 velocity=3.141592653589793
- joint r_hj_middle_3: limit lower=-1.5707963267948966 upper=1.5707963267948966 effort=7.5 velocity=3.141592653589793 -> lower=0 upper=1.5708 effort=7.5 velocity=3.141592653589793
- joint r_hj_middle_4: limit lower=-1.5707963267948966 upper=1.5707963267948966 effort=7.5 velocity=3.141592653589793 -> lower=0 upper=1.5708 effort=7.5 velocity=3.141592653589793
- joint r_hj_pinky_1: limit lower=-0.017453292519943295 upper=1.0471975511965976 effort=7.5 velocity=3.141592653589793 -> lower=-0.0174533 upper=0.16 effort=7.5 velocity=3.141592653589793
- joint r_hj_pinky_3: limit lower=-1.5707963267948966 upper=1.5707963267948966 effort=7.5 velocity=3.141592653589793 -> lower=0 upper=1.5708 effort=7.5 velocity=3.141592653589793
- joint r_hj_pinky_4: limit lower=-1.5707963267948966 upper=1.5707963267948966 effort=7.5 velocity=3.141592653589793 -> lower=0 upper=1.5708 effort=7.5 velocity=3.141592653589793
- joint r_hj_ring_1: limit lower=-0.6108652381980153 upper=0.4188790204786391 effort=7.5 velocity=3.141592653589793 -> lower=-0.16 upper=0.16 effort=7.5 velocity=3.141592653589793
- joint r_hj_ring_3: limit lower=-1.5707963267948966 upper=1.5707963267948966 effort=7.5 velocity=3.141592653589793 -> lower=0 upper=1.5708 effort=7.5 velocity=3.141592653589793
- joint r_hj_ring_4: limit lower=-1.5707963267948966 upper=1.5707963267948966 effort=7.5 velocity=3.141592653589793 -> lower=0 upper=1.5708 effort=7.5 velocity=3.141592653589793
- joint r_hj_thumb_3: limit lower=-1.5707963267948966 upper=1.5707963267948966 effort=7.5 velocity=3.141592653589793 -> lower=0 upper=1.05 effort=7.5 velocity=3.141592653589793
- joint r_hj_thumb_4: limit lower=-1.5707963267948966 upper=1.5707963267948966 effort=7.5 velocity=3.141592653589793 -> lower=0 upper=1.05 effort=7.5 velocity=3.141592653589793
