Commit message: feat(dg5f-m): 손 관절 사양을 벤더 **공식 매뉴얼**로 교체 — effort·velocity·가동범위
출처: `DG5F_User_Manual_En_v1.1.4` §3.1(전기 사양) · §3.3.1(모터별 가동범위).
벤더가 같은 값을 두 곳에서 다르게 준다 — 드라이버 URDF 와 매뉴얼이 어긋난다:

  effort    URDF 7.5 N·m     → 매뉴얼 peak(stall) **2.0 N·m**      (3.75배 과대)
  velocity  URDF 3.142 rad/s → 매뉴얼 무부하 75 RPM = **7.854**     (2.5배 과소)
  가동범위   7개 관절 불일치. 대표적으로 thumb_1 URDF -22~+51° vs 매뉴얼 -22~+77°

URDF 의 7.5 와 π 는 placeholder 로 보인다(20관절이 전부 같은 값, π 라는 우연). 매뉴얼은
제품 사양서이고 CAD 릴리스와도 일치한다(엄지 상한 CAD 1.3439 rad = 77°).

★가장 큰 것: **엄지 대향이 ±9.2° 로 잘려 있었다**(매뉴얼 -22~+77° 의 19%). 엄지가 손가락
  쪽으로 돌아오지 못하면 인벨롭 파지가 원리적으로 불가능하다. 09.09 "감싸지 못한다" 의
  유력한 원인이고, 힘·armature 문제가 아니었다(매뉴얼 인벨롭 정격 10kg / 최대 20kg —
  134g 컵을 못 감싸는 것이 힘 문제일 수 없다).

- `JOINT_LIMIT_RESTRICTIONS`(좁히기 전용) → `HAND_JOINT_SPEC`(절대값 설정)으로 교체.
  매뉴얼 값이 URDF 보다 **넓은** 관절이 있어 좁히기로는 옮길 수 없었다.
- 좌우 미러는 **원본 URDF 의 좌우 관계에서 판정**한다. 표를 그대로 양손에 적용하면
  `l_hj_thumb_2` 가 [0,+3.14]→[-2.71,0] 로 부호가 뒤집힌다(작업 중 실제로 한 번 만들었다).
- 과신전(`_3/_4` 음수)은 자산에서 **허용**한다 — 실기가 실제로 된다. 정책이 명령하지
  못하게 막는 것은 프로필 `hand_action_limit_override` 몫이고, 물리 한계와 액션 범위는
  다른 층이다(09.09 사용자 확정).
- 미등록 자산은 빌드 에러. 나머지 4자산은 아직 매뉴얼 대조 전이라 None 으로 선언.

⚠매뉴얼 연속 정격은 **0.4 N·m** 이고 2.0 은 스톨(순간)이다. 매뉴얼이 스톨 연속 사용에
  "급격한 온도 상승·제품 손상"을 경고하므로 파지 유지 토크는 별도로 감시할 것.

계약 테스트 5종 추가: 사양표 선언 강제 · effort/velocity 반영 · 매뉴얼 가동범위 반영 ·
엄지 대향 가동폭 회귀 방지 · 좌우 미러 보존. urdf 도구 테스트 142개 통과.

Co-Authored-By: Claude Opus 5 <noreply@anthropic.com>
Claude-Session: https://claude.ai/code/session_01X3UjBxvcdQMDLsryR8e6J6

File: generated/fabric/openarm_dg5f-m_bi_left/openarm_dg5f-m_bi_left.urdf (robot description, URDF)
Before this commit: robot openarm_dg5f-m_bi_left, 62 links, 61 joints
Joints:
- joint rj_dg_1_1: limit lower=-0.16 upper=0.16 effort=7.5 velocity=3.1415927 -> lower=-1.3439 upper=0.383972 effort=7.5 velocity=3.1415927
- joint rj_dg_1_2: limit lower=-0 upper=3.14159265 effort=7.5 velocity=3.1415927 -> lower=-0 upper=2.70526 effort=7.5 velocity=3.1415927
- joint rj_dg_1_3: limit lower=0 upper=1.05 effort=7.5 velocity=3.1415927 -> lower=-1.5708 upper=1.5708 effort=7.5 velocity=3.1415927
- joint rj_dg_1_4: limit lower=0 upper=1.05 effort=7.5 velocity=3.1415927 -> lower=-1.5708 upper=1.5708 effort=7.5 velocity=3.1415927
- joint rj_dg_2_1: limit lower=-0.16 upper=0.16 effort=7.5 velocity=3.1415927 -> lower=-0.349066 upper=0.541052 effort=7.5 velocity=3.1415927
- joint rj_dg_2_2: limit lower=-0 upper=2.00712864 effort=7.5 velocity=3.1415927 -> lower=0 upper=2.00713 effort=7.5 velocity=3.1415927
- joint rj_dg_2_3: limit lower=0 upper=1.5708 effort=7.5 velocity=3.1415927 -> lower=-1.5708 upper=1.5708 effort=7.5 velocity=3.1415927
- joint rj_dg_2_4: limit lower=0 upper=1.5708 effort=7.5 velocity=3.1415927 -> lower=-1.5708 upper=1.5708 effort=7.5 velocity=3.1415927
- joint rj_dg_3_1: limit lower=-0.16 upper=0.16 effort=7.5 velocity=3.1415927 -> lower=-0.523599 upper=0.523599 effort=7.5 velocity=3.1415927
- joint rj_dg_3_2: limit lower=-0 upper=1.95476876 effort=7.5 velocity=3.1415927 -> lower=0 upper=2.00713 effort=7.5 velocity=3.1415927
- joint rj_dg_3_3: limit lower=0 upper=1.5708 effort=7.5 velocity=3.1415927 -> lower=-1.5708 upper=1.5708 effort=7.5 velocity=3.1415927
- joint rj_dg_3_4: limit lower=0 upper=1.5708 effort=7.5 velocity=3.1415927 -> lower=-1.5708 upper=1.5708 effort=7.5 velocity=3.1415927
- joint rj_dg_4_1: limit lower=-0.16 upper=0.16 effort=7.5 velocity=3.1415927 -> lower=-0.558505 upper=0.261799 effort=7.5 velocity=3.1415927
- joint rj_dg_4_2: limit lower=-0 upper=1.90240888 effort=7.5 velocity=3.1415927 -> lower=0 upper=1.91986 effort=7.5 velocity=3.1415927
- joint rj_dg_4_3: limit lower=0 upper=1.5708 effort=7.5 velocity=3.1415927 -> lower=-1.5708 upper=1.5708 effort=7.5 velocity=3.1415927
- joint rj_dg_4_4: limit lower=0 upper=1.5708 effort=7.5 velocity=3.1415927 -> lower=-1.5708 upper=1.5708 effort=7.5 velocity=3.1415927
- joint rj_dg_5_1: limit lower=-0.16 upper=0.0174533 effort=7.5 velocity=3.1415927 -> lower=-1.0472 upper=-0 effort=7.5 velocity=3.1415927
- joint rj_dg_5_2: limit lower=-0.610865238 upper=0.41887902 effort=7.5 velocity=3.1415927 -> lower=-1.5708 upper=0.261799 effort=7.5 velocity=3.1415927
- joint rj_dg_5_3: limit lower=0 upper=1.5708 effort=7.5 velocity=3.1415927 -> lower=-1.5708 upper=1.5708 effort=7.5 velocity=3.1415927
- joint rj_dg_5_4: limit lower=0 upper=1.5708 effort=7.5 velocity=3.1415927 -> lower=-1.5708 upper=1.5708 effort=7.5 velocity=3.1415927

File: generated/fabric/openarm_dg5f-m_bi_right/openarm_dg5f-m_bi_right.urdf (robot description, URDF)
Before this commit: robot openarm_dg5f-m_bi_right, 62 links, 61 joints
Joints:
- joint rj_dg_1_1: limit lower=-0.16 upper=0.16 effort=7.5 velocity=3.1415927 -> lower=-0.383972 upper=1.3439 effort=7.5 velocity=3.1415927
- joint rj_dg_1_2: limit lower=-3.14159265 upper=0 effort=7.5 velocity=3.1415927 -> lower=-2.70526 upper=0 effort=7.5 velocity=3.1415927
- joint rj_dg_1_3: limit lower=0 upper=1.05 effort=7.5 velocity=3.1415927 -> lower=-1.5708 upper=1.5708 effort=7.5 velocity=3.1415927
- joint rj_dg_1_4: limit lower=0 upper=1.05 effort=7.5 velocity=3.1415927 -> lower=-1.5708 upper=1.5708 effort=7.5 velocity=3.1415927
- joint rj_dg_2_1: limit lower=-0.16 upper=0.16 effort=7.5 velocity=3.1415927 -> lower=-0.541052 upper=0.349066 effort=7.5 velocity=3.1415927
- joint rj_dg_2_2: limit lower=-0 upper=2.00712864 effort=7.5 velocity=3.1415927 -> lower=0 upper=2.00713 effort=7.5 velocity=3.1415927
- joint rj_dg_2_3: limit lower=0 upper=1.5708 effort=7.5 velocity=3.1415927 -> lower=-1.5708 upper=1.5708 effort=7.5 velocity=3.1415927
- joint rj_dg_2_4: limit lower=0 upper=1.5708 effort=7.5 velocity=3.1415927 -> lower=-1.5708 upper=1.5708 effort=7.5 velocity=3.1415927
- joint rj_dg_3_1: limit lower=-0.16 upper=0.16 effort=7.5 velocity=3.1415927 -> lower=-0.523599 upper=0.523599 effort=7.5 velocity=3.1415927
- joint rj_dg_3_2: limit lower=-0 upper=1.95476876 effort=7.5 velocity=3.1415927 -> lower=0 upper=2.00713 effort=7.5 velocity=3.1415927
- joint rj_dg_3_3: limit lower=0 upper=1.5708 effort=7.5 velocity=3.1415927 -> lower=-1.5708 upper=1.5708 effort=7.5 velocity=3.1415927
- joint rj_dg_3_4: limit lower=0 upper=1.5708 effort=7.5 velocity=3.1415927 -> lower=-1.5708 upper=1.5708 effort=7.5 velocity=3.1415927
- joint rj_dg_4_1: limit lower=-0.16 upper=0.16 effort=7.5 velocity=3.1415927 -> lower=-0.261799 upper=0.558505 effort=7.5 velocity=3.1415927
- joint rj_dg_4_2: limit lower=-0 upper=1.90240888 effort=7.5 velocity=3.1415927 -> lower=0 upper=1.91986 effort=7.5 velocity=3.1415927
- joint rj_dg_4_3: limit lower=0 upper=1.5708 effort=7.5 velocity=3.1415927 -> lower=-1.5708 upper=1.5708 effort=7.5 velocity=3.1415927
- joint rj_dg_4_4: limit lower=0 upper=1.5708 effort=7.5 velocity=3.1415927 -> lower=-1.5708 upper=1.5708 effort=7.5 velocity=3.1415927
- joint rj_dg_5_1: limit lower=-0.0174533 upper=0.16 effort=7.5 velocity=3.1415927 -> lower=0 upper=1.0472 effort=7.5 velocity=3.1415927
- joint rj_dg_5_2: limit lower=-0.41887902 upper=0.610865238 effort=7.5 velocity=3.1415927 -> lower=-0.261799 upper=1.5708 effort=7.5 velocity=3.1415927
- joint rj_dg_5_3: limit lower=0 upper=1.5708 effort=7.5 velocity=3.1415927 -> lower=-1.5708 upper=1.5708 effort=7.5 velocity=3.1415927
- joint rj_dg_5_4: limit lower=0 upper=1.5708 effort=7.5 velocity=3.1415927 -> lower=-1.5708 upper=1.5708 effort=7.5 velocity=3.1415927

File: generated/rl/openarm_dg5f-m_bi_rl.urdf (robot description, URDF)
Before this commit: robot openarm_dg5f_m_bi_rl, 80 links, 79 joints
Joints:
- joint l_hj_index_1: limit lower=-0.16 upper=0.16 effort=7.5 velocity=3.141592653589793 -> lower=-0.349066 upper=0.541052 effort=2 velocity=7.854
- joint l_hj_index_2: limit lower=-0.0 upper=2.007128639793479 effort=7.5 velocity=3.141592653589793 -> lower=0 upper=2.00713 effort=2 velocity=7.854
- joint l_hj_index_3: limit lower=0 upper=1.5708 effort=7.5 velocity=3.141592653589793 -> lower=-1.5708 upper=1.5708 effort=2 velocity=7.854
- joint l_hj_index_4: limit lower=0 upper=1.5708 effort=7.5 velocity=3.141592653589793 -> lower=-1.5708 upper=1.5708 effort=2 velocity=7.854
- joint l_hj_middle_1: limit lower=-0.16 upper=0.16 effort=7.5 velocity=3.141592653589793 -> lower=-0.523599 upper=0.523599 effort=2 velocity=7.854
- joint l_hj_middle_2: limit lower=-0.0 upper=1.9547687622336491 effort=7.5 velocity=3.141592653589793 -> lower=0 upper=2.00713 effort=2 velocity=7.854
- joint l_hj_middle_3: limit lower=0 upper=1.5708 effort=7.5 velocity=3.141592653589793 -> lower=-1.5708 upper=1.5708 effort=2 velocity=7.854
- joint l_hj_middle_4: limit lower=0 upper=1.5708 effort=7.5 velocity=3.141592653589793 -> lower=-1.5708 upper=1.5708 effort=2 velocity=7.854
- joint l_hj_pinky_1: limit lower=-0.16 upper=0.0174533 effort=7.5 velocity=3.141592653589793 -> lower=-1.0472 upper=-0 effort=2 velocity=7.854
- joint l_hj_pinky_2: limit lower=-0.6108652381980153 upper=0.4188790204786391 effort=7.5 velocity=3.141592653589793 -> lower=-1.5708 upper=0.261799 effort=2 velocity=7.854
- joint l_hj_pinky_3: limit lower=0 upper=1.5708 effort=7.5 velocity=3.141592653589793 -> lower=-1.5708 upper=1.5708 effort=2 velocity=7.854
- joint l_hj_pinky_4: limit lower=0 upper=1.5708 effort=7.5 velocity=3.141592653589793 -> lower=-1.5708 upper=1.5708 effort=2 velocity=7.854
- joint l_hj_ring_1: limit lower=-0.16 upper=0.16 effort=7.5 velocity=3.141592653589793 -> lower=-0.558505 upper=0.261799 effort=2 velocity=7.854
- joint l_hj_ring_2: limit lower=-0.0 upper=1.9024088846738192 effort=7.5 velocity=3.141592653589793 -> lower=0 upper=1.91986 effort=2 velocity=7.854
- joint l_hj_ring_3: limit lower=0 upper=1.5708 effort=7.5 velocity=3.141592653589793 -> lower=-1.5708 upper=1.5708 effort=2 velocity=7.854
- joint l_hj_ring_4: limit lower=0 upper=1.5708 effort=7.5 velocity=3.141592653589793 -> lower=-1.5708 upper=1.5708 effort=2 velocity=7.854
- joint l_hj_thumb_1: limit lower=-0.16 upper=0.16 effort=7.5 velocity=3.141592653589793 -> lower=-1.3439 upper=0.383972 effort=2 velocity=7.854
- joint l_hj_thumb_2: limit lower=-0.0 upper=3.141592653589793 effort=7.5 velocity=3.141592653589793 -> lower=-0 upper=2.70526 effort=2 velocity=7.854
- joint l_hj_thumb_3: limit lower=0 upper=1.05 effort=7.5 velocity=3.141592653589793 -> lower=-1.5708 upper=1.5708 effort=2 velocity=7.854
- joint l_hj_thumb_4: limit lower=0 upper=1.05 effort=7.5 velocity=3.141592653589793 -> lower=-1.5708 upper=1.5708 effort=2 velocity=7.854
- joint r_hj_index_1: limit lower=-0.16 upper=0.16 effort=7.5 velocity=3.141592653589793 -> lower=-0.541052 upper=0.349066 effort=2 velocity=7.854
- joint r_hj_index_2: limit lower=-0.0 upper=2.007128639793479 effort=7.5 velocity=3.141592653589793 -> lower=0 upper=2.00713 effort=2 velocity=7.854
- joint r_hj_index_3: limit lower=0 upper=1.5708 effort=7.5 velocity=3.141592653589793 -> lower=-1.5708 upper=1.5708 effort=2 velocity=7.854
- joint r_hj_index_4: limit lower=0 upper=1.5708 effort=7.5 velocity=3.141592653589793 -> lower=-1.5708 upper=1.5708 effort=2 velocity=7.854
- joint r_hj_middle_1: limit lower=-0.16 upper=0.16 effort=7.5 velocity=3.141592653589793 -> lower=-0.523599 upper=0.523599 effort=2 velocity=7.854
- joint r_hj_middle_2: limit lower=-0.0 upper=1.9547687622336491 effort=7.5 velocity=3.141592653589793 -> lower=0 upper=2.00713 effort=2 velocity=7.854
- joint r_hj_middle_3: limit lower=0 upper=1.5708 effort=7.5 velocity=3.141592653589793 -> lower=-1.5708 upper=1.5708 effort=2 velocity=7.854
- joint r_hj_middle_4: limit lower=0 upper=1.5708 effort=7.5 velocity=3.141592653589793 -> lower=-1.5708 upper=1.5708 effort=2 velocity=7.854
- joint r_hj_pinky_1: limit lower=-0.0174533 upper=0.16 effort=7.5 velocity=3.141592653589793 -> lower=0 upper=1.0472 effort=2 velocity=7.854
- joint r_hj_pinky_2: limit lower=-0.4188790204786391 upper=0.6108652381980153 effort=7.5 velocity=3.141592653589793 -> lower=-0.261799 upper=1.5708 effort=2 velocity=7.854
- joint r_hj_pinky_3: limit lower=0 upper=1.5708 effort=7.5 velocity=3.141592653589793 -> lower=-1.5708 upper=1.5708 effort=2 velocity=7.854
- joint r_hj_pinky_4: limit lower=0 upper=1.5708 effort=7.5 velocity=3.141592653589793 -> lower=-1.5708 upper=1.5708 effort=2 velocity=7.854
- joint r_hj_ring_1: limit lower=-0.16 upper=0.16 effort=7.5 velocity=3.141592653589793 -> lower=-0.261799 upper=0.558505 effort=2 velocity=7.854
- joint r_hj_ring_2: limit lower=-0.0 upper=1.9024088846738192 effort=7.5 velocity=3.141592653589793 -> lower=0 upper=1.91986 effort=2 velocity=7.854
- joint r_hj_ring_3: limit lower=0 upper=1.5708 effort=7.5 velocity=3.141592653589793 -> lower=-1.5708 upper=1.5708 effort=2 velocity=7.854
- joint r_hj_ring_4: limit lower=0 upper=1.5708 effort=7.5 velocity=3.141592653589793 -> lower=-1.5708 upper=1.5708 effort=2 velocity=7.854
- joint r_hj_thumb_1: limit lower=-0.16 upper=0.16 effort=7.5 velocity=3.141592653589793 -> lower=-0.383972 upper=1.3439 effort=2 velocity=7.854
- joint r_hj_thumb_2: limit lower=-3.141592653589793 upper=0.0 effort=7.5 velocity=3.141592653589793 -> lower=-2.70526 upper=0 effort=2 velocity=7.854
- joint r_hj_thumb_3: limit lower=0 upper=1.05 effort=7.5 velocity=3.141592653589793 -> lower=-1.5708 upper=1.5708 effort=2 velocity=7.854
- joint r_hj_thumb_4: limit lower=0 upper=1.05 effort=7.5 velocity=3.141592653589793 -> lower=-1.5708 upper=1.5708 effort=2 velocity=7.854
