Commit message: feat: dg5f-m-short 에 OpenArm 플랜지 어댑터 판 추가
vendor/dg5f_m_short_adaptor 의 메시를 팔 플랜지(link7)와 손 마운트 **사이**에 넣는다
(사용자 지시 09.10). short 는 마운트/베이스 구간이 짧아 플랜지에 직접 물리지 않는다.

기하: 55 x 55 x 10 mm 평판(메시 mm 단위 -> scale 0.001). 결합면 z=0 팔 쪽 / z=10 손 쪽.
      체인: r_al_7 -(z 0.0495)-> r_hl_flange_adapter -(z 0.010)-> r_hl_adapter -> ...
      결과 palm 이 10.00mm 밀렸다(dg5f-m 대비 47.30 -> 37.30mm).

⚠질량 0.06912 kg 은 **벤더값이 아니다** — 벤더가 재질·질량을 안 줘서 메시 부피
  25.600 cm^3(바운딩박스 충전율 84.6%)에 알루미늄 6061 을 곱한 추정이다. 관성도 같은
  메시로 적분(대각, com z 4.986mm). 물리 링크는 질량이 없으면 PhysX 에서 1kg 유령이
  되므로 넣지 않을 수 없다(§0 의 명시적 예외). 벤더가 실제 값을 주면 교체할 것.

★hand_mount_parent_links 를 **체인 추적**으로 고쳤다. 마운트 조인트의 부모가 더 이상
  항상 팔 플랜지가 아니다 — 직접 부모만 보던 구 판본은 어댑터 삽입 후 빈 집합을 돌려
  strip_stock_gripper_motor 와 make_self_collision_safe 가 **둘 다 no-op** 이 됐고,
  link7 이 스톡 그리퍼 모터와 볼트 collision 을 유지해 감사가 8건 실패했다
  (최대 24.5mm 관통). 이제 어댑터가 몇 개 끼어도 견딘다. 감사 재통과(0 fail).

테스트: mount flush 검사를 "팔 플랜지가 부모인 조인트"로 일반화하고, 중간 어댑터는
        두께만 더해야 한다(횡변위·회전 0)는 조건을 추가. 벤더 손 질량 합에서
        `*_hl_flange_adapter` 제외(추정값이 섞이면 드리프트 검사가 무의미).
        어댑터 존재·질량·두께 전용 테스트 신설. 144 passed.

Co-Authored-By: Claude Opus 5 <noreply@anthropic.com>
Claude-Session: https://claude.ai/code/session_01X3UjBxvcdQMDLsryR8e6J6

File: assemblies/openarm_modular_dual_tesollo_short.xacro (robot description, xacro)
@@ -19,4 +19,6 @@
   <!-- External dependencies -->
   <xacro:include filename="$(find openarm_description)/urdf/robot/openarm_robot.xacro"/>
+  <!-- DG-5F-M-short <-> OpenArm 플랜지 어댑터 판(사용자 지시 09.10) -->
+  <xacro:include filename="../eef/dg5f_m_short_adaptor.xacro"/>
   <!-- Tesollo wrappers -->
   <xacro:include filename="../eef/tesollo_left_wrapper.xacro"/>
@@ -78,8 +80,14 @@
     palm_com_xyz="$(arg left_palm_ee_xyz)"
   />
-  <joint name="mount_left_link7_to_tesollo" type="fixed">
+  <xacro:dg5f_m_short_adaptor prefix="left_"/>
+  <joint name="mount_left_link7_to_adaptor" type="fixed">
     <parent link="openarm_left_link7"/>
+    <child  link="left_dg5f_short_adaptor"/>
+    <origin xyz="$(arg left_mount_xyz)" rpy="$(arg left_mount_rpy)"/>
+  </joint>
+  <joint name="mount_left_adaptor_to_tesollo" type="fixed">
+    <parent link="left_dg5f_short_adaptor"/>
     <child  link="left_base_link"/>
-    <origin xyz="$(arg left_mount_xyz)" rpy="$(arg left_mount_rpy)"/>
+    <origin xyz="0 0 ${dg5f_short_adaptor_thickness}" rpy="0 0 0"/>
   </joint>
   <!-- RIGHT: Tesollo right hand on openarm_right_link7 -->
@@ -89,8 +97,17 @@
     palm_com_xyz="$(arg right_palm_ee_xyz)"
   />
-  <joint name="mount_right_link7_to_tesollo" type="fixed">
+  <!-- ★09.10 어댑터 판을 플랜지와 손 마운트 **사이**에 끼운다. 회전은 종전과 같은
+       자리(플랜지->어댑터)에 두고, 어댑터->손은 판 두께 10mm 만 더한다. 판은 55x55
+       정사각이라 z 회전은 기하에 영향이 없다. 결과로 손이 플랜지에서 10mm 멀어진다. -->
+  <xacro:dg5f_m_short_adaptor prefix="right_"/>
+  <joint name="mount_right_link7_to_adaptor" type="fixed">
     <parent link="openarm_right_link7"/>
-    <child  link="right_base_link"/>
+    <child  link="right_dg5f_short_adaptor"/>
     <origin xyz="$(arg right_mount_xyz)" rpy="$(arg right_mount_rpy)"/>
   </joint>
+  <joint name="mount_right_adaptor_to_tesollo" type="fixed">
+    <parent link="right_dg5f_short_adaptor"/>
+    <child  link="right_base_link"/>
+    <origin xyz="0 0 ${dg5f_short_adaptor_thickness}" rpy="0 0 0"/>
+  </joint>
 </robot>

File: generated/fabric/openarm_dg5f-m-short_bi_left/openarm_dg5f-m-short_bi_left.urdf (robot description, URDF)
Before this commit: robot openarm_dg5f-m-short_bi_left, 62 links, 61 joints
Joints:
- joint palm_link_joint: origin xyz=0 -3e-07 0.076 rpy=0 0 1.5707964 -> xyz=0 -3e-07 0.086 rpy=0 0 1.5707964
- joint rj_dg_1_1: limit lower=-1.34390352 upper=0.383972435 effort=7.5 velocity=3.1415927 -> lower=-1.3439 upper=0.383972 effort=7.5 velocity=3.1415927
- joint rj_dg_1_2: limit lower=-0 upper=2.70526034 effort=7.5 velocity=3.1415927 -> lower=-0 upper=2.70526 effort=7.5 velocity=3.1415927
- joint rj_dg_1_3: limit lower=-1.57079633 upper=1.57079633 effort=7.5 velocity=3.1415927 -> lower=-1.5708 upper=1.5708 effort=7.5 velocity=3.1415927
- joint rj_dg_1_4: limit lower=-1.57079633 upper=1.57079633 effort=7.5 velocity=3.1415927 -> lower=-1.5708 upper=1.5708 effort=7.5 velocity=3.1415927
- joint rj_dg_2_1: limit lower=-0.34906585 upper=0.541052068 effort=7.5 velocity=3.1415927 -> lower=-0.349066 upper=0.541052 effort=7.5 velocity=3.1415927
- joint rj_dg_2_2: limit lower=-0 upper=2.00712864 effort=7.5 velocity=3.1415927 -> lower=0 upper=2.00713 effort=7.5 velocity=3.1415927
- joint rj_dg_2_3: limit lower=-1.57079633 upper=1.57079633 effort=7.5 velocity=3.1415927 -> lower=-1.5708 upper=1.5708 effort=7.5 velocity=3.1415927
- joint rj_dg_2_4: limit lower=-1.57079633 upper=1.57079633 effort=7.5 velocity=3.1415927 -> lower=-1.5708 upper=1.5708 effort=7.5 velocity=3.1415927
- joint rj_dg_3_1: limit lower=-0.436332313 upper=0.436332313 effort=7.5 velocity=3.1415927 -> lower=-0.436332 upper=0.436332 effort=7.5 velocity=3.1415927
- joint rj_dg_3_2: limit lower=0 upper=2.00712864 effort=7.5 velocity=3.1415927 -> lower=0 upper=2.00713 effort=7.5 velocity=3.1415927
- joint rj_dg_3_3: limit lower=-1.57079633 upper=1.57079633 effort=7.5 velocity=3.1415927 -> lower=-1.5708 upper=1.5708 effort=7.5 velocity=3.1415927
- joint rj_dg_3_4: limit lower=-1.57079633 upper=1.57079633 effort=7.5 velocity=3.1415927 -> lower=-1.5708 upper=1.5708 effort=7.5 velocity=3.1415927
- joint rj_dg_4_1: limit lower=-0.558505361 upper=0.261799388 effort=7.5 velocity=3.1415927 -> lower=-0.558505 upper=0.261799 effort=7.5 velocity=3.1415927
- joint rj_dg_4_2: limit lower=0 upper=1.91986218 effort=7.5 velocity=3.1415927 -> lower=0 upper=1.91986 effort=7.5 velocity=3.1415927
- joint rj_dg_4_3: limit lower=-1.57079633 upper=1.57079633 effort=7.5 velocity=3.1415927 -> lower=-1.5708 upper=1.5708 effort=7.5 velocity=3.1415927
- joint rj_dg_4_4: limit lower=-1.57079633 upper=1.57079633 effort=7.5 velocity=3.1415927 -> lower=-1.5708 upper=1.5708 effort=7.5 velocity=3.1415927
- joint rj_dg_5_1: limit lower=-1.04719755 upper=0 effort=7.5 velocity=3.1415927 -> lower=-1.0472 upper=-0 effort=7.5 velocity=3.1415927
- joint rj_dg_5_2: limit lower=-1.57079633 upper=0.261799388 effort=7.5 velocity=3.1415927 -> lower=-1.5708 upper=0.261799 effort=7.5 velocity=3.1415927
- joint rj_dg_5_3: limit lower=-1.57079633 upper=1.57079633 effort=7.5 velocity=3.1415927 -> lower=-1.5708 upper=1.5708 effort=7.5 velocity=3.1415927
- joint rj_dg_5_4: limit lower=-1.57079633 upper=1.57079633 effort=7.5 velocity=3.1415927 -> lower=-1.5708 upper=1.5708 effort=7.5 velocity=3.1415927

File: generated/fabric/openarm_dg5f-m-short_bi_right/openarm_dg5f-m-short_bi_right.urdf (robot description, URDF)
Before this commit: robot openarm_dg5f-m-short_bi_right, 62 links, 61 joints
Joints:
- joint palm_link_joint: origin xyz=0 3e-07 0.076 rpy=0. 0. -1.5707964 -> xyz=0 3e-07 0.086 rpy=0. 0. -1.5707964
- joint rj_dg_1_1: limit lower=-0.383972435 upper=1.34390352 effort=7.5 velocity=3.1415927 -> lower=-0.383972 upper=1.3439 effort=7.5 velocity=3.1415927
- joint rj_dg_1_2: limit lower=-2.70526034 upper=0 effort=7.5 velocity=3.1415927 -> lower=-2.70526 upper=0 effort=7.5 velocity=3.1415927
- joint rj_dg_1_3: limit lower=-1.57079633 upper=1.57079633 effort=7.5 velocity=3.1415927 -> lower=-1.5708 upper=1.5708 effort=7.5 velocity=3.1415927
- joint rj_dg_1_4: limit lower=-1.57079633 upper=1.57079633 effort=7.5 velocity=3.1415927 -> lower=-1.5708 upper=1.5708 effort=7.5 velocity=3.1415927
- joint rj_dg_2_1: limit lower=-0.541052068 upper=0.34906585 effort=7.5 velocity=3.1415927 -> lower=-0.541052 upper=0.349066 effort=7.5 velocity=3.1415927
- joint rj_dg_2_2: limit lower=-0 upper=2.00712864 effort=7.5 velocity=3.1415927 -> lower=0 upper=2.00713 effort=7.5 velocity=3.1415927
- joint rj_dg_2_3: limit lower=-1.57079633 upper=1.57079633 effort=7.5 velocity=3.1415927 -> lower=-1.5708 upper=1.5708 effort=7.5 velocity=3.1415927
- joint rj_dg_2_4: limit lower=-1.57079633 upper=1.57079633 effort=7.5 velocity=3.1415927 -> lower=-1.5708 upper=1.5708 effort=7.5 velocity=3.1415927
- joint rj_dg_3_1: limit lower=-0.436332313 upper=0.436332313 effort=7.5 velocity=3.1415927 -> lower=-0.436332 upper=0.436332 effort=7.5 velocity=3.1415927
- joint rj_dg_3_2: limit lower=0 upper=2.00712864 effort=7.5 velocity=3.1415927 -> lower=0 upper=2.00713 effort=7.5 velocity=3.1415927
- joint rj_dg_3_3: limit lower=-1.57079633 upper=1.57079633 effort=7.5 velocity=3.1415927 -> lower=-1.5708 upper=1.5708 effort=7.5 velocity=3.1415927
- joint rj_dg_3_4: limit lower=-1.57079633 upper=1.57079633 effort=7.5 velocity=3.1415927 -> lower=-1.5708 upper=1.5708 effort=7.5 velocity=3.1415927
- joint rj_dg_4_1: limit lower=-0.261799388 upper=0.558505361 effort=7.5 velocity=3.1415927 -> lower=-0.261799 upper=0.558505 effort=7.5 velocity=3.1415927
- joint rj_dg_4_2: limit lower=0 upper=1.91986218 effort=7.5 velocity=3.1415927 -> lower=0 upper=1.91986 effort=7.5 velocity=3.1415927
- joint rj_dg_4_3: limit lower=-1.57079633 upper=1.57079633 effort=7.5 velocity=3.1415927 -> lower=-1.5708 upper=1.5708 effort=7.5 velocity=3.1415927
- joint rj_dg_4_4: limit lower=-1.57079633 upper=1.57079633 effort=7.5 velocity=3.1415927 -> lower=-1.5708 upper=1.5708 effort=7.5 velocity=3.1415927
- joint rj_dg_5_1: limit lower=-0 upper=1.04719755 effort=7.5 velocity=3.1415927 -> lower=0 upper=1.0472 effort=7.5 velocity=3.1415927
- joint rj_dg_5_2: limit lower=-0.261799388 upper=1.57079633 effort=7.5 velocity=3.1415927 -> lower=-0.261799 upper=1.5708 effort=7.5 velocity=3.1415927
- joint rj_dg_5_3: limit lower=-1.57079633 upper=1.57079633 effort=7.5 velocity=3.1415927 -> lower=-1.5708 upper=1.5708 effort=7.5 velocity=3.1415927
- joint rj_dg_5_4: limit lower=-1.57079633 upper=1.57079633 effort=7.5 velocity=3.1415927 -> lower=-1.5708 upper=1.5708 effort=7.5 velocity=3.1415927

File: generated/fabric/openarm_dg5f-m_bi_left/openarm_dg5f-m_bi_left.urdf (robot description, URDF)
Before this commit: robot openarm_dg5f-m_bi_left, 62 links, 61 joints
Joints:
- joint rj_dg_3_1: limit lower=-0.523599 upper=0.523599 effort=7.5 velocity=3.1415927 -> lower=-0.436332 upper=0.436332 effort=7.5 velocity=3.1415927

File: generated/fabric/openarm_dg5f-m_bi_right/openarm_dg5f-m_bi_right.urdf (robot description, URDF)
Before this commit: robot openarm_dg5f-m_bi_right, 62 links, 61 joints
Joints:
- joint rj_dg_3_1: limit lower=-0.523599 upper=0.523599 effort=7.5 velocity=3.1415927 -> lower=-0.436332 upper=0.436332 effort=7.5 velocity=3.1415927

File: generated/fabric/openarm_dg5f-s_bi_left/openarm_dg5f-s_bi_left.urdf (robot description, URDF)
Before this commit: robot openarm_dg5f-s_bi_left, 62 links, 61 joints
Joints:
- joint rj_dg_1_1: limit lower=-1.57079633 upper=1.57079633 effort=7.5 velocity=3.1415927 -> lower=-1.5708 upper=1.5708 effort=7.5 velocity=3.1415927
- joint rj_dg_1_2: limit lower=0 upper=2.67035376 effort=7.5 velocity=3.1415927 -> lower=-0 upper=2.67035 effort=7.5 velocity=3.1415927
- joint rj_dg_1_3: limit lower=-1.57079633 upper=1.57079633 effort=7.5 velocity=3.1415927 -> lower=-1.5708 upper=1.5708 effort=7.5 velocity=3.1415927
- joint rj_dg_1_4: limit lower=-1.57079633 upper=1.57079633 effort=7.5 velocity=3.1415927 -> lower=-1.5708 upper=1.5708 effort=7.5 velocity=3.1415927
- joint rj_dg_2_1: limit lower=-0.261799388 upper=0.837758041 effort=7.5 velocity=3.1415927 -> lower=-0.261799 upper=0.837758 effort=7.5 velocity=3.1415927
- joint rj_dg_2_2: limit lower=0 upper=2.19911486 effort=7.5 velocity=3.1415927 -> lower=0 upper=2.19911 effort=7.5 velocity=3.1415927
- joint rj_dg_2_3: limit lower=-1.57079633 upper=1.57079633 effort=7.5 velocity=3.1415927 -> lower=-1.5708 upper=1.5708 effort=7.5 velocity=3.1415927
- joint rj_dg_2_4: limit lower=-1.57079633 upper=1.57079633 effort=7.5 velocity=3.1415927 -> lower=-1.5708 upper=1.5708 effort=7.5 velocity=3.1415927
- joint rj_dg_3_1: limit lower=-0.733038286 upper=0.575958653 effort=7.5 velocity=3.1415927 -> lower=-0.733038 upper=0.575959 effort=7.5 velocity=3.1415927
- joint rj_dg_3_2: limit lower=0 upper=2.26892803 effort=7.5 velocity=3.1415927 -> lower=0 upper=2.26893 effort=7.5 velocity=3.1415927
- joint rj_dg_3_3: limit lower=-1.57079633 upper=1.57079633 effort=7.5 velocity=3.1415927 -> lower=-1.5708 upper=1.5708 effort=7.5 velocity=3.1415927
- joint rj_dg_3_4: limit lower=-1.57079633 upper=1.57079633 effort=7.5 velocity=3.1415927 -> lower=-1.5708 upper=1.5708 effort=7.5 velocity=3.1415927
- joint rj_dg_4_1: limit lower=-0.837758041 upper=0.20943951 effort=7.5 velocity=3.1415927 -> lower=-0.837758 upper=0.20944 effort=7.5 velocity=3.1415927
- joint rj_dg_4_2: limit lower=0 upper=2.21656815 effort=7.5 velocity=3.1415927 -> lower=0 upper=2.21657 effort=7.5 velocity=3.1415927
- joint rj_dg_4_3: limit lower=-1.57079633 upper=1.57079633 effort=7.5 velocity=3.1415927 -> lower=-1.5708 upper=1.5708 effort=7.5 velocity=3.1415927
- joint rj_dg_4_4: limit lower=-1.57079633 upper=1.57079633 effort=7.5 velocity=3.1415927 -> lower=-1.5708 upper=1.5708 effort=7.5 velocity=3.1415927
- joint rj_dg_5_1: limit lower=-1.04719755 upper=0 effort=7.5 velocity=3.1415927 -> lower=-1.0472 upper=-0 effort=7.5 velocity=3.1415927
- joint rj_dg_5_2: limit lower=-1.57079633 upper=0.645771823 effort=7.5 velocity=3.1415927 -> lower=-1.5708 upper=0.645772 effort=7.5 velocity=3.1415927
- joint rj_dg_5_3: limit lower=-1.57079633 upper=1.57079633 effort=7.5 velocity=3.1415927 -> lower=-1.5708 upper=1.5708 effort=7.5 velocity=3.1415927
- joint rj_dg_5_4: limit lower=-1.57079633 upper=1.57079633 effort=7.5 velocity=3.1415927 -> lower=-1.5708 upper=1.5708 effort=7.5 velocity=3.1415927

File: generated/fabric/openarm_dg5f-s_bi_right/openarm_dg5f-s_bi_right.urdf (robot description, URDF)
Before this commit: robot openarm_dg5f-s_bi_right, 62 links, 61 joints
Joints:
- joint rj_dg_1_1: limit lower=-1.57079633 upper=1.57079633 effort=7.5 velocity=3.1415927 -> lower=-1.5708 upper=1.5708 effort=7.5 velocity=3.1415927
- joint rj_dg_1_2: limit lower=-2.67035376 upper=0 effort=7.5 velocity=3.1415927 -> lower=-2.67035 upper=0 effort=7.5 velocity=3.1415927
- joint rj_dg_1_3: limit lower=-1.57079633 upper=1.57079633 effort=7.5 velocity=3.1415927 -> lower=-1.5708 upper=1.5708 effort=7.5 velocity=3.1415927
- joint rj_dg_1_4: limit lower=-1.57079633 upper=1.57079633 effort=7.5 velocity=3.1415927 -> lower=-1.5708 upper=1.5708 effort=7.5 velocity=3.1415927
- joint rj_dg_2_1: limit lower=-0.837758041 upper=0.261799388 effort=7.5 velocity=3.1415927 -> lower=-0.837758 upper=0.261799 effort=7.5 velocity=3.1415927
- joint rj_dg_2_2: limit lower=0 upper=2.19911486 effort=7.5 velocity=3.1415927 -> lower=0 upper=2.19911 effort=7.5 velocity=3.1415927
- joint rj_dg_2_3: limit lower=-1.57079633 upper=1.57079633 effort=7.5 velocity=3.1415927 -> lower=-1.5708 upper=1.5708 effort=7.5 velocity=3.1415927
- joint rj_dg_2_4: limit lower=-1.57079633 upper=1.57079633 effort=7.5 velocity=3.1415927 -> lower=-1.5708 upper=1.5708 effort=7.5 velocity=3.1415927
- joint rj_dg_3_1: limit lower=-0.575958653 upper=0.733038286 effort=7.5 velocity=3.1415927 -> lower=-0.575959 upper=0.733038 effort=7.5 velocity=3.1415927
- joint rj_dg_3_2: limit lower=0 upper=2.26892803 effort=7.5 velocity=3.1415927 -> lower=0 upper=2.26893 effort=7.5 velocity=3.1415927
- joint rj_dg_3_3: limit lower=-1.57079633 upper=1.57079633 effort=7.5 velocity=3.1415927 -> lower=-1.5708 upper=1.5708 effort=7.5 velocity=3.1415927
- joint rj_dg_3_4: limit lower=-1.57079633 upper=1.57079633 effort=7.5 velocity=3.1415927 -> lower=-1.5708 upper=1.5708 effort=7.5 velocity=3.1415927
- joint rj_dg_4_1: limit lower=-0.20943951 upper=0.837758041 effort=7.5 velocity=3.1415927 -> lower=-0.20944 upper=0.837758 effort=7.5 velocity=3.1415927
- joint rj_dg_4_2: limit lower=0 upper=2.21656815 effort=7.5 velocity=3.1415927 -> lower=0 upper=2.21657 effort=7.5 velocity=3.1415927
- joint rj_dg_4_3: limit lower=-1.57079633 upper=1.57079633 effort=7.5 velocity=3.1415927 -> lower=-1.5708 upper=1.5708 effort=7.5 velocity=3.1415927
- joint rj_dg_4_4: limit lower=-1.57079633 upper=1.57079633 effort=7.5 velocity=3.1415927 -> lower=-1.5708 upper=1.5708 effort=7.5 velocity=3.1415927
- joint rj_dg_5_1: limit lower=0 upper=1.04719755 effort=7.5 velocity=3.1415927 -> lower=0 upper=1.0472 effort=7.5 velocity=3.1415927
- joint rj_dg_5_2: limit lower=-0.645771823 upper=1.57079633 effort=7.5 velocity=3.1415927 -> lower=-0.645772 upper=1.5708 effort=7.5 velocity=3.1415927
- joint rj_dg_5_3: limit lower=-1.57079633 upper=1.57079633 effort=7.5 velocity=3.1415927 -> lower=-1.5708 upper=1.5708 effort=7.5 velocity=3.1415927
- joint rj_dg_5_4: limit lower=-1.57079633 upper=1.57079633 effort=7.5 velocity=3.1415927 -> lower=-1.5708 upper=1.5708 effort=7.5 velocity=3.1415927

File: generated/rl/openarm_dg5f-m-short_bi_rl.urdf (robot description, URDF)
Before this commit: robot openarm_dg5f_m_short_bi_rl, 80 links, 79 joints
Links:
- added link l_hl_flange_adapter, mass 0.06912; collision mesh filename=file:///home/user/rl_ws/urdf/vendor/dg5f_m_short_adaptor/me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 scale=0.001 0.001 0.001; visual mesh filename=file:///home/user/rl_ws/urdf/vendor/dg5f_m_short_adaptor/me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 scale=0.001 0.001 0.001
- added link r_hl_flange_adapter, mass 0.06912; collision mesh filename=file:///home/user/rl_ws/urdf/vendor/dg5f_m_short_adaptor/me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 scale=0.001 0.001 0.001; visual mesh filename=file:///home/user/rl_ws/urdf/vendor/dg5f_m_short_adaptor/me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 scale=0.001 0.001 0.001
Joints:
- added joint l_hj_flange_adapter: type fixed, parent l_al_7, child l_hl_flange_adapter, origin xyz=0 0 0.0495 rpy=0 0 1.5707964
- added joint r_hj_flange_adapter: type fixed, parent r_al_7, child r_hl_flange_adapter, origin xyz=0 0.0000003 0.0495 rpy=0 0 -1.5707964
- joint l_hj_mount: origin xyz=0 0 0.0495 rpy=0 0 1.5707964 -> xyz=0 0 0.01 rpy=0 0 0; parent l_al_7 -> l_hl_flange_adapter
- joint r_hj_mount: origin xyz=0 0.0000003 0.0495 rpy=0 0 -1.5707964 -> xyz=0 0 0.01 rpy=0 0 0; parent r_al_7 -> r_hl_flange_adapter

File: generated/source/openarm_tesollo_bi_short.urdf (robot description, URDF)
Before this commit: robot openarm_dual_tesollo_short, 80 links, 79 joints
Links:
- added link left_dg5f_short_adaptor, mass 0.06912; collision mesh filename=file:///home/user/rl_ws/urdf/vendor/dg5f_m_short_adaptor/me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 scale=0.001 0.001 0.001; visual mesh filename=file:///home/user/rl_ws/urdf/vendor/dg5f_m_short_adaptor/me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 scale=0.001 0.001 0.001
- added link right_dg5f_short_adaptor, mass 0.06912; collision mesh filename=file:///home/user/rl_ws/urdf/vendor/dg5f_m_short_adaptor/me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 scale=0.001 0.001 0.001; visual mesh filename=file:///home/user/rl_ws/urdf/vendor/dg5f_m_short_adaptor/me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 scale=0.001 0.001 0.001
Joints:
- removed joint mount_left_link7_to_tesollo
- removed joint mount_right_link7_to_tesollo
- added joint mount_left_adaptor_to_tesollo: type fixed, parent left_dg5f_short_adaptor, child left_base_link, origin xyz=0 0 0.01 rpy=0 0 0
- added joint mount_left_link7_to_adaptor: type fixed, parent openarm_left_link7, child left_dg5f_short_adaptor, origin xyz=0 0 0.0495 rpy=0 0 1.5707964
- added joint mount_right_adaptor_to_tesollo: type fixed, parent right_dg5f_short_adaptor, child right_base_link, origin xyz=0 0 0.01 rpy=0 0 0
- added joint mount_right_link7_to_adaptor: type fixed, parent openarm_right_link7, child right_dg5f_short_adaptor, origin xyz=0 0.0000003 0.0495 rpy=0 0 -1.5707964
